File: PCB-Design/hardware/spb-busbar/spb-busbar.kicad_pcb (KiCad board)
At the start: 4 copper layers, 298.5 x 45 mm, 29 parts, among them J1 LEG1 DC+, J10 LEG3 DC-, J11 LEG3 DC+, J12 LEG3 DC-, J13 STACK DC+ (to level above: it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, J14 STACK DC- (to level below: it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, J15 LEVEL V: 1 DC+, 2 DC- (HV ref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, J2 LEG1 DC-, J3 LEG1 DC+, J4 LEG1 DC-, J5 LEG2 DC+, J6 LEG2 DC-, J7 LEG2 DC+, J8 LEG2 DC-, J9 LEG3 DC+

Commit message: ﻿Busbar: copper weight as argument (default 2 oz, JLCPCB JLC3313), 2/3/4 oz estimates
Other:
- board text added: "4 layers, 1.6 mm FR4, 2 oz Cu on ALL layers (JLCPCB: 2 oz outer + 2 oz inner, JLC3313 stack-up), ENIG"
- board text removed: "4 layers, 1.6 mm FR4, 70 um (2 oz) Cu on ALL layers (3 oz optional), ENIG"

Commit message: ﻿Rev B as one leg: one DC pair, one AC bolt pad (option B drivers)
- make_kicad_bb_revb.py: one DC+/DC- REDCUBE pair at the centre feeding a laminated
  terminal row (L1/L3 DC+, L2/L4 DC-) over the full width; the four AC terminals replaced
  by one M6 bolt pad (AC_BOLT_M6, 14 mm pad, via rings); two drivers, one star per pair.
  231 parts, DRC 0/0/0, routing 0 failures
- schematic regenerated, check_sch_vs_pcb: 0 problems
- busbar: one DC pair per leg (6 bolt points), DRC clean
- Q3D export/post for the new terminals; leg Q3D setup at 2 % convergence
- deck: step 8 slides for the new layout (Q3D numbers follow)
Parts:
- removed J10, J12: LEG3 DC-, spb_fab:BUS_M4_REDCUBE
- removed J11: LEG3 DC+, spb_fab:BUS_M4_REDCUBE
- removed J13: STACK DC+ (to level above: its DC-), spb_fab:BUS_LUG_M6
- removed J14: STACK DC- (to level below: its DC+), spb_fab:BUS_LUG_M6
- removed J15: LEVEL V: 1 DC+, 2 DC- (HV referenced), Connector_PinHeader_2.54mm:PinHeader_1x02_P2.54mm_Vertical
- J3: value LEG1 DC+ -> LEG2 DC+
- J4: value LEG1 DC- -> LEG2 DC-
- J5: value LEG2 DC+ -> LEG3 DC+
- J6: value LEG2 DC- -> LEG3 DC-
- J7: value LEG2 DC+ -> STACK DC+ (to level above: its DC-); footprint spb_fab:BUS_M4_REDCUBE -> spb_fab:BUS_LUG_M6
- J8: value LEG2 DC- -> STACK DC- (to level below: its DC+); footprint spb_fab:BUS_M4_REDCUBE -> spb_fab:BUS_LUG_M6
- J9: value LEG3 DC+ -> LEVEL V: 1 DC+, 2 DC- (HV referenced); footprint spb_fab:BUS_M4_REDCUBE -> Connector_PinHeader_2.54mm:PinHeader_1x02_P2.54mm_Vertical
- moved J5 118.2 mm to (248.5, 61.2)
- moved J6 118.2 mm to (260.5, 61.2)
- moved J3 70.8 mm to (154.0, 61.2)
- moved J4 70.8 mm to (166.0, 61.2)
- moved J9 67.8 mm to (160.0, 41.0)
- moved J7 34.9 mm to (148.0, 43.0)
- moved J8 25.4 mm to (172.0, 43.0)
- moved J1 23.8 mm to (59.5, 61.2)
- moved J2 23.8 mm to (71.5, 61.2)
