File: PCB-Design/hardware/spb-bb-revb/spb-bb-revb.kicad_sch (KiCad schematic)
At the start: 235 parts, among them J1 DC+, J10 U.FL L2, J11 U.FL D2, J12 DC+, J13 DC-, J14 V_ISO,HS in, J15 V_ISO,LS in, J16 CTRL2, J17 FAN 12V, J18 U.FL H3, J19 U.FL L3, J2 DC-, J20 U.FL D3, J21 U.FL H4, J22 U.FL L4, J23 U.FL D4, J24 AC, J25 AC, J26 AC, J27 AC, J28 1, J3 V_ISO,HS in, J4 V_ISO,LS in, J5 CTRL1, J6 U.FL H1, J7 U.FL L1, J8 U.FL D1, J9 U.FL H2, Q1 EPC2361, Q2 EPC2361, Q3 EPC2361, Q4 EPC2361, Q5 EPC2361, Q6 EPC2361, Q7 EPC2361, Q8 EPC2361, U1 2EDF7275K, U2 2EDF7275K

Commit message: ﻿Rev B as one leg: one DC pair, one AC bolt pad (option B drivers)
- make_kicad_bb_revb.py: one DC+/DC- REDCUBE pair at the centre feeding a laminated
  terminal row (L1/L3 DC+, L2/L4 DC-) over the full width; the four AC terminals replaced
  by one M6 bolt pad (AC_BOLT_M6, 14 mm pad, via rings); two drivers, one star per pair.
  231 parts, DRC 0/0/0, routing 0 failures
- schematic regenerated, check_sch_vs_pcb: 0 problems
- busbar: one DC pair per leg (6 bolt points), DRC clean
- Q3D export/post for the new terminals; leg Q3D setup at 2 % convergence
- deck: step 8 slides for the new layout (Q3D numbers follow)
Parts:
- removed J24, J25, J26, J27: AC, TerminalBlock_Wuerth:Wuerth_REDCUBE-THR_WP-THRBU_74650174_THR, symbol Connector_Generic:Conn_01x01
- removed J28: 1, Connector_PinHeader_2.54mm:PinHeader_1x02_P2.54mm_Vertical, symbol Connector_Generic:Conn_01x02
- J12: value DC+ -> V_ISO,HS in; footprint TerminalBlock_Wuerth:Wuerth_REDCUBE-THR_WP-THRBU_74650174_THR -> Connector_PinHeader_2.54mm:PinHeader_1x02_P2.54mm_Vertical; symbol Connector_Generic:Conn_01x01 -> Connector_Generic:Conn_01x02; MPN Wuerth 74650174 (REDCUBE THR, M4) -> 2.54 mm header 1x2
- J13: value DC- -> V_ISO,LS in; footprint TerminalBlock_Wuerth:Wuerth_REDCUBE-THR_WP-THRBU_74650174_THR -> Connector_PinHeader_2.54mm:PinHeader_1x02_P2.54mm_Vertical; symbol Connector_Generic:Conn_01x01 -> Connector_Generic:Conn_01x02; MPN Wuerth 74650174 (REDCUBE THR, M4) -> 2.54 mm header 1x2
- J14: value V_ISO,HS in -> CTRL2; footprint Connector_PinHeader_2.54mm:PinHeader_1x02_P2.54mm_Vertical -> Connector_PinHeader_2.54mm:PinHeader_2x03_P2.54mm_Vertical; symbol Connector_Generic:Conn_01x02 -> Connector_Generic:Conn_02x03_Odd_Even; MPN 2.54 mm header 1x2 -> 2.54 mm header 2x3
- J15: value V_ISO,LS in -> FAN 12V; MPN 2.54 mm header 1x2 -> 2.54 mm header 1x2 (fan)
- J16: value CTRL2 -> U.FL H3; footprint Connector_PinHeader_2.54mm:PinHeader_2x03_P2.54mm_Vertical -> spb_fab:U.FL_Hirose_U.FL-R-SMT-1_Vertical; symbol Connector_Generic:Conn_02x03_Odd_Even -> Connector:Conn_Coaxial; MPN 2.54 mm header 2x3 -> Hirose U.FL-R-SMT-1(10)
- J17: value FAN 12V -> U.FL L3; footprint Connector_PinHeader_2.54mm:PinHeader_1x02_P2.54mm_Vertical -> spb_fab:U.FL_Hirose_U.FL-R-SMT-1_Vertical; symbol Connector_Generic:Conn_01x02 -> Connector:Conn_Coaxial; MPN 2.54 mm header 1x2 (fan) -> Hirose U.FL-R-SMT-1(10)
- J18: value U.FL H3 -> U.FL D3
- J19: value U.FL L3 -> U.FL H4
- J20: value U.FL D3 -> U.FL L4
- J21: value U.FL H4 -> U.FL D4
- J22: value U.FL L4 -> AC; footprint spb_fab:U.FL_Hirose_U.FL-R-SMT-1_Vertical -> spb_fab:AC_BOLT_M6; symbol Connector:Conn_Coaxial -> Connector_Generic:Conn_01x01; MPN Hirose U.FL-R-SMT-1(10) -> M6 bolt + nut, 12 x 5 mm Cu bar
- J23: value U.FL D4 -> 1; footprint spb_fab:U.FL_Hirose_U.FL-R-SMT-1_Vertical -> Connector_PinHeader_2.54mm:PinHeader_1x02_P2.54mm_Vertical; symbol Connector:Conn_Coaxial -> Connector_Generic:Conn_01x02; MPN Hirose U.FL-R-SMT-1(10) -> 2.54 mm header 1x2
Connections:
- net +12V2: now also J15.1 (Pin_1); no longer J17.1 (Pin_1)
- net C_12V2: now also J14.1 (Pin_1); no longer J16.1 (Pin_1)
- net C_DIS2: now also J14.5 (Pin_5); no longer J16.5 (Pin_5)
- net C_GND2: now also J14.2 (Pin_2), J14.6 (Pin_6); no longer J16.2 (Pin_2), J16.6 (Pin_6)
- net C_PWMH2: now also J14.3 (Pin_3); no longer J16.3 (Pin_3)
- net C_PWML2: now also J14.4 (Pin_4); no longer J16.4 (Pin_4)
- net DCN: now also J23.2 (Pin_2); no longer J13.1 (Pin_1)
- net DCP: no longer J12.1 (Pin_1)
- net GNDI2: now also J15.2 (Pin_2); no longer J17.2 (Pin_2)
- net KH2: now also J16.2 (Ext), J19.2 (Ext); no longer J18.2 (Ext), J21.2 (Ext)
- net KL2: now also J17.2 (Ext), J20.2 (Ext); no longer J19.2 (Ext), J22.2 (Ext)
- net LSRC3: now also J18.2 (Ext); no longer J20.2 (Ext)
- net LSRC4: now also J21.2 (Ext); no longer J23.2 (Ext)
- net NTC: now also J23.1 (Pin_1)
- net SW: now also J22.1 (Pin_1)
- net VINA_N2: now also J12.2 (Pin_2); no longer J14.2 (Pin_2)
- net VINA_P2: now also J12.1 (Pin_1); no longer J14.1 (Pin_1)
- net VINB_N2: now also J13.2 (Pin_2); no longer J15.2 (Pin_2)
- net VINB_P2: now also J13.1 (Pin_1); no longer J15.1 (Pin_1)
- net at R47.2: now also J21.1 (In); no longer J23.1 (In)
- net at R44.1: now also J18.1 (In); no longer J20.1 (In)
- net at R42.1: now also J16.1 (In); no longer J18.1 (In)
- net at R46.2: now also J20.1 (In); no longer J22.1 (In)
- net at R45.2: now also J19.1 (In); no longer J21.1 (In)
- net at R43.1: now also J17.1 (In); no longer J19.1 (In)
Other:
- note added: "J12 / L6: HS block 2"
- note added: "J13 / L7: LS block 2"
- note added: "J22: AC output, M6 bolt pad, 12 x 5 mm Cu bar bolted on"
- note added: "J23 is in the LS domain (high voltage)"
- note added: "the bar passes through a LEM HO 250-S (off board,"
- note removed: "J14 / L6: HS block 2"
- note removed: "J15 / L7: LS block 2"
- note removed: "J24-J27: M4 REDCUBE AC terminals, bolted 12 x 5 mm Cu bar"
- note removed: "J28 is in the LS domain (high voltage)"
- note removed: "one output stub through a LEM HO 250-S (off board,"
- moved on the sheet: J15, J18, J19, J20, J21

Commit message: ﻿Rev B: one continuous capacitor bank on a uniform 3 mm grid
The per-block bank left an empty column at each block centre (Rev A DC entry). The bank is
now placed once for the leg: 3 rows x 25 x 10 uF 1210 at x = -36 ... +36 mm, no gaps
(75 bank + 24 bypass MLCCs). DRC 0/0/0, schematic = PCB (0 problems).
Parts:
- added C116, C117, C118, C119, C120, C121, C122, C123, C124, C125, C126, C127: 10uF 100V X7S, spb_fab:C_1210_3225Metric_TightCrtYd, symbol Device:C
- C100, C94, C97: value 4.7uF 25V X7R -> 10uF 100V X7S; footprint Capacitor_SMD:C_0805_2012Metric -> spb_fab:C_1210_3225Metric_TightCrtYd; MPN Murata GRM21BR71E475KA73 -> Murata GRM32EC72A106KE05L
- C13, C14, C15, C16: value 10uF 100V X7S -> 1uF 16V X7R; footprint spb_fab:C_1210_3225Metric_TightCrtYd -> Capacitor_SMD:C_0402_1005Metric; MPN Murata GRM32EC72A106KE05L -> Murata GRM155R71C105KA12
- C17, C18: value 10uF 100V X7S -> 100pF C0G; footprint spb_fab:C_1210_3225Metric_TightCrtYd -> Capacitor_SMD:C_0402_1005Metric; MPN Murata GRM32EC72A106KE05L -> Murata GRM1555C1H101JA01
- C19: value 10uF 100V X7S -> 22nF 25V X7R; footprint spb_fab:C_1210_3225Metric_TightCrtYd -> Capacitor_SMD:C_0402_1005Metric; MPN Murata GRM32EC72A106KE05L -> Murata GRM155R71E223KA61
- C20, C23, C26: value 10uF 100V X7S -> 4.7uF 25V X7R; footprint spb_fab:C_1210_3225Metric_TightCrtYd -> Capacitor_SMD:C_0805_2012Metric; MPN Murata GRM32EC72A106KE05L -> Murata GRM21BR71E475KA73
- C21, C22, C24, C25: value 10uF 100V X7S -> 4.7uF 16V X5R; footprint spb_fab:C_1210_3225Metric_TightCrtYd -> Capacitor_SMD:C_0603_1608Metric; MPN Murata GRM32EC72A106KE05L -> Murata GRM188R61C475KAAJ
- C27, C28, C29, C30, C31, C32, C33, C34, C35, C36: value 10uF 100V X7S -> 1uF 100V X7S; footprint spb_fab:C_1210_3225Metric_TightCrtYd -> spb_fab:C_0805_2012Metric_TightCrtYd; MPN Murata GRM32EC72A106KE05L -> TDK C2012X7S2A105K125AB
- C37, C38: value 1uF 16V X7R -> 1uF 100V X7S; footprint Capacitor_SMD:C_0402_1005Metric -> spb_fab:C_0805_2012Metric_TightCrtYd; MPN Murata GRM155R71C105KA12 -> TDK C2012X7S2A105K125AB
- C41, C42: value 100pF C0G -> 1uF 16V X7R; MPN Murata GRM1555C1H101JA01 -> Murata GRM155R71C105KA12
- C43: value 22nF 25V X7R -> 100pF C0G; MPN Murata GRM155R71E223KA61 -> Murata GRM1555C1H101JA01
- C44: value 4.7uF 25V X7R -> 100pF C0G; footprint Capacitor_SMD:C_0805_2012Metric -> Capacitor_SMD:C_0402_1005Metric; MPN Murata GRM21BR71E475KA73 -> Murata GRM1555C1H101JA01
- C45: value 4.7uF 16V X5R -> 22nF 25V X7R; footprint Capacitor_SMD:C_0603_1608Metric -> Capacitor_SMD:C_0402_1005Metric; MPN Murata GRM188R61C475KAAJ -> Murata GRM155R71E223KA61
- C46, C49: value 4.7uF 16V X5R -> 4.7uF 25V X7R; footprint Capacitor_SMD:C_0603_1608Metric -> Capacitor_SMD:C_0805_2012Metric; MPN Murata GRM188R61C475KAAJ -> Murata GRM21BR71E475KA73
- C47, C50: value 4.7uF 25V X7R -> 4.7uF 16V X5R; footprint Capacitor_SMD:C_0805_2012Metric -> Capacitor_SMD:C_0603_1608Metric; MPN Murata GRM21BR71E475KA73 -> Murata GRM188R61C475KAAJ
- C51: value 1uF 100V X7S -> 4.7uF 16V X5R; footprint spb_fab:C_0805_2012Metric_TightCrtYd -> Capacitor_SMD:C_0603_1608Metric; MPN TDK C2012X7S2A105K125AB -> Murata GRM188R61C475KAAJ
- C52: value 1uF 100V X7S -> 4.7uF 25V X7R; footprint spb_fab:C_0805_2012Metric_TightCrtYd -> Capacitor_SMD:C_0805_2012Metric; MPN TDK C2012X7S2A105K125AB -> Murata GRM21BR71E475KA73
- C53, C54, C55, C56, C57, C58, C59, C60, C61, C62: value 1uF 100V X7S -> 10uF 100V X7S; footprint spb_fab:C_0805_2012Metric_TightCrtYd -> spb_fab:C_1210_3225Metric_TightCrtYd; MPN TDK C2012X7S2A105K125AB -> Murata GRM32EC72A106KE05L
- C87, C88, C89, C90: value 1uF 16V X7R -> 10uF 100V X7S; footprint Capacitor_SMD:C_0402_1005Metric -> spb_fab:C_1210_3225Metric_TightCrtYd; MPN Murata GRM155R71C105KA12 -> Murata GRM32EC72A106KE05L
- C91, C92: value 100pF C0G -> 10uF 100V X7S; footprint Capacitor_SMD:C_0402_1005Metric -> spb_fab:C_1210_3225Metric_TightCrtYd; MPN Murata GRM1555C1H101JA01 -> Murata GRM32EC72A106KE05L
- C93: value 22nF 25V X7R -> 10uF 100V X7S; footprint Capacitor_SMD:C_0402_1005Metric -> spb_fab:C_1210_3225Metric_TightCrtYd; MPN Murata GRM155R71E223KA61 -> Murata GRM32EC72A106KE05L
- C95, C96, C98, C99: value 4.7uF 16V X5R -> 10uF 100V X7S; footprint Capacitor_SMD:C_0603_1608Metric -> spb_fab:C_1210_3225Metric_TightCrtYd; MPN Murata GRM188R61C475KAAJ -> Murata GRM32EC72A106KE05L
Connections:
- net +12V1: now also C26.1; no longer C50.1
- net +12V2: now also C52.1; no longer C100.1
- net DCN: now also C100.2, C101.2, C102.2, C106.1, C107.1, C108.1, C109.1, C110.1, C29.2, C30.2, C31.2, C32.2, C33.2, C34.2, C35.2, C36.2, C37.2, C38.2, C53.1, C54.1, C55.1, C56.1, C57.1, C58.1, C59.1, C60.1, C61.1, C62.1, C71.1, C72.1, C73.1, C74.1, C75.1, C76.1, C77.1, C79.2, C80.2, C81.2, C82.2, C83.2, C84.2, C85.2, C86.2, C87.2, C88.2, C89.2, C90.2, C91.2, C92.2, C93.2, C94.2, C95.2, C96.2, C97.2, C98.2, C99.2, C116.1, C117.1, C118.1, C119.1, C120.1, C121.1, C122.1, C123.1, C124.1, C125.1, C126.1, C127.1; no longer C101.1, C102.1, C106.2, C107.2, C108.2, C109.2, C110.2, C13.1, C14.1, C15.1, C16.1, C17.1, C18.1, C19.1, C20.1, C21.2, C22.2, C23.2, C24.2, C25.2, C26.2, C29.1, C30.1, C31.1, C32.1, C33.1, C34.1, C35.1, C36.1, C51.2, C52.2, C53.2, C54.2, C55.2, C56.2, C57.2, C58.2, C59.2, C60.2, C61.2, C62.2, C71.2, C72.2, C73.2, C74.2, C75.2, C76.2, C77.2, C79.1, C80.1, C81.1, C82.1, C83.1, C84.1, C85.1, C86.1
- net DCP: now also C100.1, C101.1, C102.1, C106.2, C107.2, C108.2, C109.2, C110.2, C29.1, C30.1, C31.1, C32.1, C33.1, C34.1, C35.1, C36.1, C37.1, C38.1, C53.2, C54.2, C55.2, C56.2, C57.2, C58.2, C59.2, C60.2, C61.2, C62.2, C71.2, C72.2, C73.2, C74.2, C75.2, C76.2, C77.2, C79.1, C80.1, C81.1, C82.1, C83.1, C84.1, C85.1, C86.1, C87.1, C88.1, C89.1, C90.1, C91.1, C92.1, C93.1, C94.1, C95.1, C96.1, C97.1, C98.1, C99.1, C116.2, C117.2, C118.2, C119.2, C120.2, C121.2, C122.2, C123.2, C124.2, C125.2, C126.2, C127.2; no longer C101.2, C102.2, C106.1, C107.1, C108.1, C109.1, C110.1, C13.2, C14.2, C15.2, C16.2, C17.2, C18.2, C19.2, C20.2, C21.1, C22.1, C23.1, C24.1, C25.1, C26.1, C29.2, C30.2, C31.2, C32.2, C33.2, C34.2, C35.2, C36.2, C51.1, C52.1, C53.1, C54.1, C55.1, C56.1, C57.1, C58.1, C59.1, C60.1, C61.1, C62.1, C71.1, C72.1, C73.1, C74.1, C75.1, C76.1, C77.1, C79.2, C80.2, C81.2, C82.2, C83.2, C84.2, C85.2, C86.2
- net GNDI1: now also C17.1, C18.2, C19.2, C26.2; no longer C41.1, C42.2, C43.2, C50.2
- net GNDI2: now also C43.1, C44.2, C45.2, C52.2; no longer C100.2, C91.1, C92.2, C93.2
- net KH1: now also C13.1, C14.1, C21.1, C22.1; no longer C37.1, C38.1, C45.1, C46.1
- net KH2: now also C39.1, C40.1, C47.1, C48.1; no longer C87.1, C88.1, C95.1, C96.1
- net KL1: now also C15.2, C16.2, C24.1, C25.2; no longer C39.2, C40.2, C48.1, C49.2
- net KL2: now also C41.2, C42.2, C50.1, C51.2; no longer C89.2, C90.2, C98.1, C99.2
- net VDDA1: now also C13.2, C20.2, C21.2; no longer C37.2, C44.2, C45.2
- net VDDA2: now also C39.2, C46.2, C47.2; no longer C87.2, C94.2, C95.2
- net VDDB1: now also C16.1, C23.2, C25.1; no longer C40.1, C47.2, C49.1
- net VDDB2: now also C42.1, C49.2, C51.1; no longer C90.1, C97.2, C99.1
- net VEEA1: now also C14.2, C20.1, C22.2; no longer C38.2, C44.1, C46.2
- net VEEA2: now also C40.2, C46.1, C48.2; no longer C88.2, C94.1, C96.2
- net VEEB1: now also C15.1, C23.1, C24.2; no longer C39.1, C47.1, C48.2
- net VEEB2: now also C41.1, C49.1, C50.2; no longer C89.1, C97.1, C98.2
- net at R35.2, U2.2 (INA): now also C43.2; no longer C91.2
- net at R36.2, U2.3 (INB): now also C44.1; no longer C92.1
- net at R37.2, U2.7 (VDDI): now also C45.1; no longer C93.1
- net at R11.2, U1.2 (INA): now also C17.2; no longer C41.2
- net at R13.2, U1.7 (VDDI): now also C19.1; no longer C43.1
- net at R12.2, U1.3 (INB): now also C18.1; no longer C42.1
Other:
- note added: "DC link, 99 capacitors: 75 x 10uF 100V X7S, 24 x 1uF 100V X7S (1 uF 0805: bypass at the HS drains of each cell; 10 uF 1210: bank)"
- note removed: "DC link, 87 capacitors: 63 x 10uF 100V X7S, 24 x 1uF 100V X7S (1 uF 0805: bypass at the HS drains of each cell; 10 uF 1210: bank)"
- moved on the sheet: C10, C100, C101, C102, C103, C104, C105, C106, C107, C108, C109, C11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

Commit message: ﻿Rev B: TDK 22 uF 2220 bank (3 % ripple) and 10 bypass caps per cell
- bank: 20 x TDK C5750X7S2A226M280KB in two rows on new strips (row B 12 next to the
  cells, row A 8 clear of the DC terminal pins): 127 uF effective per leg at 75 V,
  2.9 % ripple at 50 kHz with the three legs of a level sharing the bus
- bypass: 6 x 0805 1 uF on top (loop unchanged) + 4 on the bottom per cell (L4 islands on
  the existing through vias), mirrored positions so all four cells are identical
- bb_geometry.build() accepts row overrides (Rev A unchanged)
- DRC 0/0/0, schematic = PCB (0 problems); Q3D export with bottom bypass groups;
  post-processing with the measured C at 75 V; deck: sizing, selection, bypass slides
Parts:
- removed C100, C101, C102, C103, C104, C105, C106, C107, C108, C109, C110, C111, C112, C113, C114, C115, C116, C117, C118, C119, C120, C121, C122, C123, C124, C125, C126, C127, C89, C90, C91, C92, C93, C94, C95, C96, C97, C98, C99: 10uF 100V X7S, spb_fab:C_1210_3225Metric_TightCrtYd, symbol Device:C
- C39, C40, C41, C42: value 1uF 16V X7R -> 1uF 100V X7S; footprint Capacitor_SMD:C_0402_1005Metric -> spb_fab:C_0805_2012Metric_TightCrtYd; MPN Murata GRM155R71C105KA12 -> TDK C2012X7S2A105K125AB
- C43, C44: value 100pF C0G -> 1uF 100V X7S; footprint Capacitor_SMD:C_0402_1005Metric -> spb_fab:C_0805_2012Metric_TightCrtYd; MPN Murata GRM1555C1H101JA01 -> TDK C2012X7S2A105K125AB
- C45: value 22nF 25V X7R -> 1uF 100V X7S; footprint Capacitor_SMD:C_0402_1005Metric -> spb_fab:C_0805_2012Metric_TightCrtYd; MPN Murata GRM155R71E223KA61 -> TDK C2012X7S2A105K125AB
- C46: value 4.7uF 25V X7R -> 1uF 100V X7S; footprint Capacitor_SMD:C_0805_2012Metric -> spb_fab:C_0805_2012Metric_TightCrtYd; MPN Murata GRM21BR71E475KA73 -> TDK C2012X7S2A105K125AB
- C47, C48, C50: value 4.7uF 16V X5R -> 1uF 16V X7R; footprint Capacitor_SMD:C_0603_1608Metric -> Capacitor_SMD:C_0402_1005Metric; MPN Murata GRM188R61C475KAAJ -> Murata GRM155R71C105KA12
- C49: value 4.7uF 25V X7R -> 1uF 16V X7R; footprint Capacitor_SMD:C_0805_2012Metric -> Capacitor_SMD:C_0402_1005Metric; MPN Murata GRM21BR71E475KA73 -> Murata GRM155R71C105KA12
- C51: value 4.7uF 16V X5R -> 100pF C0G; footprint Capacitor_SMD:C_0603_1608Metric -> Capacitor_SMD:C_0402_1005Metric; MPN Murata GRM188R61C475KAAJ -> Murata GRM1555C1H101JA01
- C52: value 4.7uF 25V X7R -> 100pF C0G; footprint Capacitor_SMD:C_0805_2012Metric -> Capacitor_SMD:C_0402_1005Metric; MPN Murata GRM21BR71E475KA73 -> Murata GRM1555C1H101JA01
- C53: value 10uF 100V X7S -> 22nF 25V X7R; footprint spb_fab:C_1210_3225Metric_TightCrtYd -> Capacitor_SMD:C_0402_1005Metric; MPN Murata GRM32EC72A106KE05L -> Murata GRM155R71E223KA61
- C54, C57, C60: value 10uF 100V X7S -> 4.7uF 25V X7R; footprint spb_fab:C_1210_3225Metric_TightCrtYd -> Capacitor_SMD:C_0805_2012Metric; MPN Murata GRM32EC72A106KE05L -> Murata GRM21BR71E475KA73
- C55, C56, C58, C59: value 10uF 100V X7S -> 4.7uF 16V X5R; footprint spb_fab:C_1210_3225Metric_TightCrtYd -> Capacitor_SMD:C_0603_1608Metric; MPN Murata GRM32EC72A106KE05L -> Murata GRM188R61C475KAAJ
- C61, C62, C63, C64, C65, C66, C67, C68: value 10uF 100V X7S -> 1uF 100V X7S; footprint spb_fab:C_1210_3225Metric_TightCrtYd -> spb_fab:C_0805_2012Metric_TightCrtYd; MPN Murata GRM32EC72A106KE05L -> TDK C2012X7S2A105K125AB
- C69, C70, C71, C72, C73, C74, C75, C76, C77, C78, C79, C80, C81, C82, C83, C84, C85, C86, C87, C88: value 10uF 100V X7S -> 22uF 100V X7S 2220; footprint spb_fab:C_1210_3225Metric_TightCrtYd -> spb_fab:C_2220_5750Metric_TightCrtYd; MPN Murata GRM32EC72A106KE05L -> TDK C5750X7S2A226M280KB
Connections:
- net +12V2: now also C60.1; no longer C52.1
- net DCN: now also C27.1, C28.1, C29.1, C30.1, C31.1, C32.1, C33.1, C34.1, C39.2, C40.2, C41.2, C42.2, C43.2, C44.2, C45.2, C46.2, C78.1, C79.1, C80.1, C81.1, C82.1, C83.1, C84.1, C85.1, C86.1, C87.1, C88.1; no longer C27.2, C28.2, C29.2, C30.2, C31.2, C32.2, C33.2, C34.2, C53.1, C54.1, C55.1, C56.1, C57.1, C58.1, C59.1, C60.1, C78.2, C79.2, C80.2, C81.2, C82.2, C83.2, C84.2, C85.2, C86.2, C87.2, C88.2
- net DCP: now also C27.2, C28.2, C29.2, C30.2, C31.2, C32.2, C33.2, C34.2, C39.1, C40.1, C41.1, C42.1, C43.1, C44.1, C45.1, C46.1, C78.2, C79.2, C80.2, C81.2, C82.2, C83.2, C84.2, C85.2, C86.2, C87.2, C88.2; no longer C27.1, C28.1, C29.1, C30.1, C31.1, C32.1, C33.1, C34.1, C53.2, C54.2, C55.2, C56.2, C57.2, C58.2, C59.2, C60.2, C78.1, C79.1, C80.1, C81.1, C82.1, C83.1, C84.1, C85.1, C86.1, C87.1, C88.1
- net GNDI2: now also C51.1, C53.2, C60.2; no longer C43.1, C44.2, C45.2
- net KH2: now also C55.1, C56.1; no longer C39.1, C40.1
- net KL2: now also C49.2, C50.2, C58.1, C59.2; no longer C41.2, C42.2, C50.1, C51.2
- net VDDA2: now also C54.2, C55.2; no longer C39.2, C46.2
- net VDDB2: now also C50.1, C57.2, C59.1; no longer C42.1, C49.2, C51.1
- net VEEA2: now also C54.1, C56.2; no longer C40.2, C46.1
- net VEEB2: now also C57.1, C58.2; no longer C41.1, C50.2
- net at R37.2, U2.7 (VDDI): now also C53.1; no longer C45.1
- net at R35.2, U2.2 (INA): now also C51.2; no longer C43.2
- net at R36.2, U2.3 (INB): now also C52.1; no longer C44.1
Other:
- note added: "DC link, 60 capacitors: 40 x 1uF 100V X7S, 20 x 22uF 100V X7S 2220 (1 uF 0805: bypass at the HS drains of each cell; 10 uF 1210: bank)"
- note removed: "DC link, 99 capacitors: 75 x 10uF 100V X7S, 24 x 1uF 100V X7S (1 uF 0805: bypass at the HS drains of each cell; 10 uF 1210: bank)"
- moved on the sheet: C27, C28, C29, C30, C31, C32, C33, C34, C39, C40, C41, C42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
