File: PCB-Design/hardware/spb-bb-revb/spb-bb-revb.kicad_sch (KiCad schematic)
At the start: 203 parts, among them J1 DC+, J10 U.FL L2, J11 U.FL D2, J12 V_ISO,HS in, J13 V_ISO,LS in, J14 CTRL2, J15 FAN 12V, J16 U.FL H3, J17 U.FL L3, J18 U.FL D3, J19 U.FL H4, J2 DC-, J20 U.FL L4, J21 U.FL D4, J22 AC, J23 1, J3 V_ISO,HS in, J4 V_ISO,LS in, J5 CTRL1, J6 U.FL H1, J7 U.FL L1, J8 U.FL D1, J9 U.FL H2, Q1 EPC2361, Q2 EPC2361, Q3 EPC2361, Q4 EPC2361, Q5 EPC2361, Q6 EPC2361, Q7 EPC2361, Q8 EPC2361, U1 2EDF7275K, U2 2EDF7275K

Commit message: Rev B: 3D models for every part, board STEP, design-flow deck with final loop results
- make_3d_models_revb.py: box models (STEP + VRML) for 2EDF7275K, PMK UFCS, TDK 2220 (2.8 mm),
  WE-CNSW 1206, M6 AC bolt + Cu bar, LAM 4 + spreader; parts with project models move to spb_fab
- board STEP export (fab/spb-bb-revb.step); DRC 0/0/0, schematic = PCB
- render_3d_revb.py: 3D views for the deck from the KiCad models
- deck (44 slides): Rev B bypass figure, 3D slides, fast-loop Q3D results (0.69 nH with shunt,
  0.41 nH without, cells symmetric), shunt study, symmetry cause/fix; old full-board/busbar Q3D marked
Parts:
- L1, L10, L2, L3, L4, L5, L6, L7, L8, L9: footprint Inductor_SMD:L_CommonMode_Wurth_WE-CNSW-1206 -> spb_fab:L_CommonMode_Wurth_WE-CNSW-1206
Changed lines of the file:
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@@
   (property "Reference" "L1" (at 83.82 283.21 0) (effects (font (size 1.27 1.27))))
   (property "Value" "WE-CNSW 744232601" (at 83.82 297.18 0) (effects (font (size 1.27 1.27))))
-  (property "Footprint" "Inductor_SMD:L_CommonMode_Wurth_WE-CNSW-1206" (at 83.82 289.56 0) (effects (font (size 1.27 1.27)) hide))
+  (property "Footprint" "spb_fab:L_CommonMode_Wurth_WE-CNSW-1206" (at 83.82 289.56 0) (effects (font (size 1.27 1.27)) hide))
   (property "Datasheet" "~" (at 83.82 289.56 0) (effects (font (size 1.27 1.27)) hide))
   (property "MPN" "Wurth 744232601 (600 Ohm @ 100 MHz, 260 mA)" (at 83.82 289.56 0) (effects (font (size 1.27 1.27)) hide))
@@
   (property "Reference" "L10" (at 492.76 242.57 0) (effects (font (size 1.27 1.27))))
   (property "Value" "WE-CNSW 744232601" (at 492.76 256.54 0) (effects (font (size 1.27 1.27))))
-  (property "Footprint" "Inductor_SMD:L_CommonMode_Wurth_WE-CNSW-1206" (at 492.76 248.92 0) (effects (font (size 1.27 1.27)) hide))
+  (property "Footprint" "spb_fab:L_CommonMode_Wurth_WE-CNSW-1206" (at 492.76 248.92 0) (effects (font (size 1.27 1.27)) hide))
   (property "Datasheet" "~" (at 492.76 248.92 0) (effects (font (size 1.27 1.27)) hide))
   (property "MPN" "Wurth 744232601 (600 Ohm @ 100 MHz, 260 mA)" (at 492.76 248.92 0) (effects (font (size 1.27 1.27)) hide))
@@
   (property "Reference" "L2" (at 287.02 283.21 0) (effects (font (size 1.27 1.27))))
   (property "Value" "WE-CNSW 744232601" (at 287.02 297.18 0) (effects (font (size 1.27 1.27))))
-  (property "Footprint" "Inductor_SMD:L_CommonMode_Wurth_WE-CNSW-1206" (at 287.02 289.56 0) (effects (font (size 1.27 1.27)) hide))
+  (property "Footprint" "spb_fab:L_CommonMode_Wurth_WE-CNSW-1206" (at 287.02 289.56 0) (effects (font (size 1.27 1.27)) hide))
   (property "Datasheet" "~" (at 287.02 289.56 0) (effects (font (size 1.27 1.27)) hide))
   (property "MPN" "Wurth 744232601 (600 Ohm @ 100 MHz, 260 mA)" (at 287.02 289.56 0) (effects (font (size 1.27 1.27)) hide))
@@
   (property "Reference" "L3" (at 86.36 194.31 0) (effects (font (size 1.27 1.27))))
   (property "Value" "WE-CNSW 744232601" (at 86.36 208.28 0) (effects (font (size 1.27 1.27))))
-  (property "Footprint" "Inductor_SMD:L_CommonMode_Wurth_WE-CNSW-1206" (at 86.36 200.66 0) (effects (font (size 1.27 1.27)) hide))
+  (property "Footprint" "spb_fab:L_CommonMode_Wurth_WE-CNSW-1206" (at 86.36 200.66 0) (effects (font (size 1.27 1.27)) hide))
   (property "Datasheet" "~" (at 86.36 200.66 0) (effects (font (size 1.27 1.27)) hide))
   (property "MPN" "Wurth 744232601 (600 Ohm @ 100 MHz, 260 mA)" (at 86.36 200.66 0) (effects (font (size 1.27 1.27)) hide))
@@
   (property "Reference" "L4" (at 86.36 222.25 0) (effects (font (size 1.27 1.27))))
   (property "Value" "WE-CNSW 744232601" (at 86.36 236.22 0) (effects (font (size 1.27 1.27))))
-  (property "Footprint" "Inductor_SMD:L_CommonMode_Wurth_WE-CNSW-1206" (at 86.36 228.60 0) (effects (font (size 1.27 1.27)) hide))
+  (property "Footprint" "spb_fab:L_CommonMode_Wurth_WE-CNSW-1206" (at 86.36 228.60 0) (effects (font (size 1.27 1.27)) hide))
   (property "Datasheet" "~" (at 86.36 228.60 0) (effects (font (size 1.27 1.27)) hide))
   (property "MPN" "Wurth 744232601 (600 Ohm @ 100 MHz, 260 mA)" (at 86.36 228.60 0) (effects (font (size 1.27 1.27)) hide))
@@
   (property "Reference" "L5" (at 86.36 242.57 0) (effects (font (size 1.27 1.27))))
   (property "Value" "WE-CNSW 744232601" (at 86.36 256.54 0) (effects (font (size 1.27 1.27))))
-  (property "Footprint" "Inductor_SMD:L_CommonMode_Wurth_WE-CNSW-1206" (at 86.36 248.92 0) (effects (font (size 1.27 1.27)) hide))
+  (property "Footprint" "spb_fab:L_CommonMode_Wurth_WE-CNSW-1206" (at 86.36 248.92 0) (effects (font (size 1.27 1.27)) hide))
   (property "Datasheet" "~" (at 86.36 248.92 0) (effects (font (size 1.27 1.27)) hide))
   (property "MPN" "Wurth 744232601 (600 Ohm @ 100 MHz, 260 mA)" (at 86.36 248.92 0) (effects (font (size 1.27 1.27)) hide))
@@
   (property "Reference" "L6" (at 490.22 283.21 0) (effects (font (size 1.27 1.27))))
   (property "Value" "WE-CNSW 744232601" (at 490.22 297.18 0) (effects (font (size 1.27 1.27))))
-  (property "Footprint" "Inductor_SMD:L_CommonMode_Wurth_WE-CNSW-1206" (at 490.22 289.56 0) (effects (font (size 1.27 1.27)) hide))
+  (property "Footprint" "spb_fab:L_CommonMode_Wurth_WE-CNSW-1206" (at 490.22 289.56 0) (effects (font (size 1.27 1.27)) hide))
   (property "Datasheet" "~" (at 490.22 289.56 0) (effects (font (size 1.27 1.27)) hide))
   (property "MPN" "Wurth 744232601 (600 Ohm @ 100 MHz, 260 mA)" (at 490.22 289.56 0) (effects (font (size 1.27 1.27)) hide))
@@
   (property "Reference" "L7" (at 693.42 283.21 0) (effects (font (size 1.27 1.27))))
   (property "Value" "WE-CNSW 744232601" (at 693.42 297.18 0) (effects (font (size 1.27 1.27))))
-  (property "Footprint" "Inductor_SMD:L_CommonMode_Wurth_WE-CNSW-1206" (at 693.42 289.56 0) (effects (font (size 1.27 1.27)) hide))
+  (property "Footprint" "spb_fab:L_CommonMode_Wurth_WE-CNSW-1206" (at 693.42 289.56 0) (effects (font (size 1.27 1.27)) hide))
   (property "Datasheet" "~" (at 693.42 289.56 0) (effects (font (size 1.27 1.27)) hide))
   (property "MPN" "Wurth 744232601 (600 Ohm @ 100 MHz, 260 mA)" (at 693.42 289.56 0) (effects (font (size 1.27 1.27)) hide))
@@
   (property "Reference" "L8" (at 492.76 194.31 0) (effects (font (size 1.27 1.27))))
   (property "Value" "WE-CNSW 744232601" (at 492.76 208.28 0) (effects (font (size 1.27 1.27))))
-  (property "Footprint" "Inductor_SMD:L_CommonMode_Wurth_WE-CNSW-1206" (at 492.76 200.66 0) (effects (font (size 1.27 1.27)) hide))
+  (property "Footprint" "spb_fab:L_CommonMode_Wurth_WE-CNSW-1206" (at 492.76 200.66 0) (effects (font (size 1.27 1.27)) hide))
   (property "Datasheet" "~" (at 492.76 200.66 0) (effects (font (size 1.27 1.27)) hide))
   (property "MPN" "Wurth 744232601 (600 Ohm @ 100 MHz, 260 mA)" (at 492.76 200.66 0) (effects (font (size 1.27 1.27)) hide))
@@
   (property "Reference" "L9" (at 492.76 222.25 0) (effects (font (size 1.27 1.27))))
   (property "Value" "WE-CNSW 744232601" (at 492.76 236.22 0) (effects (font (size 1.27 1.27))))
-  (property "Footprint" "Inductor_SMD:L_CommonMode_Wurth_WE-CNSW-1206" (at 492.76 228.60 0) (effects (font (size 1.27 1.27)) hide))
+  (property "Footprint" "spb_fab:L_CommonMode_Wurth_WE-CNSW-1206" (at 492.76 228.60 0) (effects (font (size 1.27 1.27)) hide))
   (property "Datasheet" "~" (at 492.76 228.60 0) (effects (font (size 1.27 1.27)) hide))
   (property "MPN" "Wurth 744232601 (600 Ohm @ 100 MHz, 260 mA)" (at 492.76 228.60 0) (effects (font (size 1.27 1.27)) hide))
