File: PCB-Design/hardware/spb-bb-revb-load/spb-bb-revb-load.kicad_sch (KiCad schematic)
At the start: 199 parts, among them J1 DC+, J10 U.FL L2, J11 U.FL D2, J12 V_ISO,HS in, J13 V_ISO,LS in, J14 CTRL2, J15 FAN 12V, J16 U.FL H3, J17 U.FL L3, J18 U.FL D3, J19 U.FL H4, J2 DC-, J20 U.FL L4, J21 U.FL D4, J22 AC, J23 1, J3 V_ISO,HS in, J4 V_ISO,LS in, J5 CTRL1, J6 U.FL H1, J7 U.FL L1, J8 U.FL D1, J9 U.FL H2, Q1 EPC2361, Q2 EPC2361, Q3 EPC2361, Q4 EPC2361, Q5 EPC2361, Q6 EPC2361, Q7 EPC2361, Q8 EPC2361, U1 2EDF7275K, U2 2EDF7275K

Commit message: Rev B boards: 1200 V control/power barrier and per-pair common-mode filtering
- Rule set in <board>.kicad_dru (exact net lists): control vs power 4.0 mm on the outer
  layers (IPC-2221B B4/A6), 3.0 mm inner (B1), 3.0 mm inside the 2EDF7275K courtyard,
  0.2 mm between the 75 V power domains. DRC 0/0 on both boards, schematic = PCB.
- Control area per block: top-layer SMD only (+ bottom GNDI plane), 4 mm / 3 mm barrier
  keepouts, nothing under the chokes and the connector on any layer.
- 2x5 SMT control header with a return next to every signal (PWM_H, PWM_L, DIS, 12 V,
  NTC), one WE-CNSW choke per pair, 12 V ferrite bead; NTC moved to the control side.
- Gate-supply islands moved outside the barrier, supplies routed on L3 around it,
  output decoupling on the bottom; AC bus/bolt 5.2 mm lower (board 89.5 x 85.2 mm).
- Removed: DC- referenced NTC header, 12 V LED, fan header (fan from the bench).
- Fab notes: IPC class 2, solder mask over all copper, all vias tented.

Co-Authored-By: Claude Opus 5.5 <noreply@anthropic.com>
Parts:
- removed D10: red, LED_SMD:LED_0603_1608Metric, symbol Device:LED
- removed J22: AC, spb_fab:AC_BOLT_M6, symbol Connector_Generic:Conn_01x01
- removed J23: 1, Connector_PinHeader_2.54mm:PinHeader_1x02_P2.54mm_Vertical, symbol Connector_Generic:Conn_01x02
- removed R50: 100k, Resistor_SMD:R_1206_3216Metric, symbol Device:R
- added FB1, FB2: BLM18PG221SN1 (220 R @ 100 MHz), Inductor_SMD:L_0603_1608Metric, symbol Device:FerriteBead
- added L11, L12, L13: WE-CNSW 744232601, spb_fab:L_CommonMode_Wurth_WE-CNSW-1206, symbol spb_fab:WE-CNSW
- C26, C60: value 4.7uF 25V X7R -> 4.7uF 25V X5R; footprint Capacitor_SMD:C_0805_2012Metric -> Capacitor_SMD:C_0603_1608Metric; MPN Murata GRM21BR71E475KA73 -> Murata GRM188R61E475KE11
- D5: value green -> PMEG3020EJ; footprint LED_SMD:LED_0603_1608Metric -> Diode_SMD:D_SOD-323F; symbol Device:LED -> Device:D_Schottky; MPN Wurth 150060GS75000 -> Nexperia PMEG3020EJ (30 V, 2 A, SOD323F)
- D7: value PMEG3020EJ -> BZX384-C5V1; footprint Diode_SMD:D_SOD-323F -> Diode_SMD:D_SOD-323; symbol Device:D_Schottky -> Device:D_Zener; MPN Nexperia PMEG3020EJ (30 V, 2 A, SOD323F) -> Nexperia BZX384-C5V1 (5.1 V, 300 mW)
- D9: value BZX384-C5V1 -> red; footprint Diode_SMD:D_SOD-323 -> LED_SMD:LED_0603_1608Metric; symbol Device:D_Zener -> Device:LED; MPN Nexperia BZX384-C5V1 (5.1 V, 300 mW) -> Wurth 150060RS75000
- J14, J5: footprint Connector_PinHeader_2.54mm:PinHeader_2x03_P2.54mm_Vertical -> spb_fab:PinHeader_2x05_P2.54mm_Vertical_SMD; symbol Connector_Generic:Conn_02x03_Odd_Even -> Connector_Generic:Conn_02x05_Odd_Even; MPN 2.54 mm header 2x3 -> Samtec TSM-105-01-T-DV (2 x 5, 2.54 mm, SMT)
- J15: value FAN 12V -> U.FL H3; footprint Connector_PinHeader_2.54mm:PinHeader_1x02_P2.54mm_Vertical -> spb_fab:U.FL_Hirose_U.FL-R-SMT-1_Vertical; symbol Connector_Generic:Conn_01x02 -> Connector:Conn_Coaxial; MPN 2.54 mm header 1x2 (fan) -> Hirose U.FL-R-SMT-1(10)
- J16: value U.FL H3 -> U.FL L3
- J17: value U.FL L3 -> U.FL D3
- J18: value U.FL D3 -> U.FL H4
- J19: value U.FL H4 -> U.FL L4
- J20: value U.FL L4 -> U.FL D4
- J21: value U.FL D4 -> AC; footprint spb_fab:U.FL_Hirose_U.FL-R-SMT-1_Vertical -> spb_fab:AC_BOLT_M6; symbol Connector:Conn_Coaxial -> Connector_Generic:Conn_01x01; MPN Hirose U.FL-R-SMT-1(10) -> M6 bolt + nut, 12 x 5 mm Cu bar
- R18: value 4.7k -> 0R; footprint Resistor_SMD:R_0603_1608Metric -> Resistor_SMD:R_0402_1005Metric; MPN 4.7k 0603 1% -> 0R 0402
- R20, R23, R43, R46: value 0R -> 953R 1%; MPN 0R 0402 -> 953R 0402 1% 100 V
- R21, R44: value 953R 1% -> 0R; MPN 953R 0402 1% 100 V -> 0R 0402
- R24: value 953R 1% -> 0R5 1%; MPN 953R 0402 1% 100 V -> 0.5R 0402 1% (Panasonic ERJ-2BQFR50X)
- R28: value 0R5 1% -> 10k 1%; MPN 0.5R 0402 1% (Panasonic ERJ-2BQFR50X) -> 10k 0402 1%
- R30: value 10k 1% -> 0R75 1%; footprint Resistor_SMD:R_0402_1005Metric -> Resistor_SMD:R_0603_1608Metric; MPN 10k 0402 1% -> 0.75R 0603 1% (Panasonic ERJ-3RQFR75V)
- R31, R33: value 0R75 1% -> 0R; footprint Resistor_SMD:R_0603_1608Metric -> Resistor_SMD:R_0402_1005Metric; MPN 0.75R 0603 1% (Panasonic ERJ-3RQFR75V) -> 0R 0402 jumper (set R_OFF here)
- R32: value 0R -> 0R75 1%; footprint Resistor_SMD:R_0402_1005Metric -> Resistor_SMD:R_0603_1608Metric; MPN 0R 0402 jumper (set R_OFF here) -> 0.75R 0603 1% (Panasonic ERJ-3RQFR75V)
- R34: value 0R -> 47R 1%; MPN 0R 0402 jumper (set R_OFF here) -> 47R 0402 1%
- R36: value 47R 1% -> 3k 1%; MPN 47R 0402 1% -> 3.0k 0402 1%
- R37: value 3k 1% -> 150R 1%; footprint Resistor_SMD:R_0402_1005Metric -> Resistor_SMD:R_0603_1608Metric; MPN 3.0k 0402 1% -> 150R 0603 1% 0.1 W
- R39: value 150R 1% -> 10k; footprint Resistor_SMD:R_0603_1608Metric -> Resistor_SMD:R_0402_1005Metric; MPN 150R 0603 1% 0.1 W -> 10k 0402 1%
- R41: value 10k -> 0R; MPN 10k 0402 1% -> 0R 0402
- R47: value 953R 1% -> 68k; footprint Resistor_SMD:R_0402_1005Metric -> Resistor_SMD:R_1206_3216Metric; MPN 953R 0402 1% 100 V -> 68k 1206 1% 200 V
- R49: value 68k -> 100k; MPN 68k 1206 1% 200 V -> 100k 1206 1% 200 V
Connections:
- net +12V1: now also C26.2, FB1.2; no longer C26.1, L3.2, R18.1
- net +12V2: now also C60.2, R36.1, FB2.2; no longer C60.1, J15.1 (Pin_1), L8.2, R37.1
- net C_12V1: now also J5.8 (Pin_8), L6.1; no longer J5.1 (Pin_1), L3.1
- net C_12V2: now also J14.8 (Pin_8), L13.1; no longer J14.1 (Pin_1), L8.1
- net C_DIS1: now also J5.6 (Pin_6), L5.4; no longer J5.5 (Pin_5), L5.1
- net C_DIS2: now also J14.6 (Pin_6), L12.4; no longer J14.5 (Pin_5), L10.1
- net C_PWMH1: now also J5.2 (Pin_2), L3.4; no longer J5.3 (Pin_3), L4.1
- net C_PWMH2: now also J14.2 (Pin_2), L10.4; no longer J14.3 (Pin_3), L9.1
- net C_PWML1: now also L4.1; no longer L4.4
- net C_PWML2: now also L11.1; no longer L9.4
- net DCN: now also D9.1 (K), J17.2 (Ext), J20.2 (Ext), R49.2; no longer J18.2 (Ext), J21.2 (Ext), RT1.1
- net DCP: now also R47.1, R49.1; no longer R48.1
- net DIS1: now also L5.3; no longer L5.2
- net DIS2: now also L12.3; no longer L10.2
- net GH_L1: now also R18.2; no longer R19.2
- net GH_L2: now also R24.1, R41.2; no longer R25.1, R42.2
- net GH_R1: now also R21.1; no longer R22.1
- net GH_R2: now also R25.2, R44.1; no longer R26.2, R45.1
- net GL_L1: now also R19.2; no longer R20.2
- net GL_L2: now also R26.1, R42.2; no longer R27.1, R43.2
- net GL_R1: now also R22.1; no longer R23.1
- net GL_R2: now also R27.2, R45.1; no longer R28.2, R46.1
- net GNDI1: now also C26.1, L3.2, L4.3, L5.2, L6.3, L7.2, R16.2, RT1.2; no longer C26.2, D5.1 (K), L3.3, R16.1
- net GNDI2: now also C60.1, L10.2, R39.2, L11.3, L12.2, L13.3; no longer C60.2, J15.2 (Pin_2), L8.3, R41.1
- net KH1: now also C22.2, R14.2; no longer C22.1, R14.1
- net KH2: now also C56.2, D7.2 (A), J15.2 (Ext), J18.2 (Ext), R28.1, R37.2; no longer C56.1, D8.2 (A), J16.2 (Ext), J19.2 (Ext), R29.1, R38.1
- net KL1: now also C24.2, C25.1, R15.2; no longer C24.1, C25.2, R15.1
- net KL2: now also C58.2, C59.1, D8.2 (A), J16.2 (Ext), J19.2 (Ext), R29.2, R38.2; no longer C58.1, C59.2, D9.2 (A), J17.2 (Ext), J20.2 (Ext), R30.2, R39.1
- net NTC: now also L7.3, RT1.1; no longer RT1.2
- net PWM_H1: now also L3.3, R16.1; no longer L4.2, R16.2
- net PWM_H2: now also L10.3, R34.1, R39.1; no longer L9.2, R35.1, R40.2
- net PWM_L1: now also L4.2; no longer L4.3
- net PWM_L2: now also R35.1, R40.2, L11.2; no longer L9.3, R36.1, R41.2
- net SW: now also J21.1 (Pin_1), R20.2, R23.1, R43.2, R46.1; no longer R21.2, R24.1, R44.2, R47.1
- net VDDA1: now also L1.4; no longer L1.2
- net VDDA2: now also D7.1 (K), L8.4; no longer D8.1 (K), L6.2
- net VDDB1: now also C25.2; no longer C25.1
- net VDDB2: now also C59.2, D8.1 (K), L9.4; no longer C59.1, D9.1 (K), L7.4
- net VEEA1: now also C22.1, L1.1, R14.1; no longer C22.2, L1.3, R14.2
- net VEEA2: now also C56.1, L8.1, R37.1; no longer C56.2, L6.3, R38.2
- net VEEB1: now also C24.1, R15.1; no longer C24.2, R15.2
- net VEEB2: now also C58.1, L9.1, R38.1; no longer C58.2, L7.1, R39.2
- net VINA_N1: now also L1.2; no longer L1.4
- net VINA_N2: now also L8.2; no longer L6.4
- net VINA_P1: now also L1.3; no longer L1.1
- net VINA_P2: now also L8.3; no longer L6.1
- net VINB_N2: now also L9.2; no longer L7.2
- net VINB_P2: now also L9.3; no longer L7.3
- net at D5.2 (A): now also R31.1; no longer R18.2
- net at R32.1: now also D6.1 (K), U2.9 (OUTB); no longer D6.2 (A)
- net at R47.2: now also R48.1; no longer J21.1 (In)
- net at J8.1 (In): now also R20.1; no longer R21.1
- net at R24.2: now also R25.1, R28.2, R30.2, R31.2; no longer J11.1 (In)
- net at C51.2, U2.2 (INA): now also R34.2; no longer R35.2
- net at C52.1, U2.3 (INB): now also R35.2; no longer R36.2
- net at J6.1 (In): now also R18.1; no longer R19.1
- net at R48.2: now also D9.2 (A); no longer R49.1
- net at J7.1 (In): now also R19.1; no longer R20.1
- net at C53.1, U2.7 (VDDI): now also R36.2; no longer R37.2
- net at R23.2: now also J11.1 (In); no longer J10.1 (In)
- net at J18.1 (In): now also R44.2; no longer R44.1
- net at R22.2: now also J10.1 (In); no longer J9.1 (In)
- removed net C_GND1: J5.2 (Pin_2), J5.6 (Pin_6), L3.4
- removed net C_GND2: J14.2 (Pin_2), J14.6 (Pin_6), L8.4
- new net: R26.2, R27.1, R29.1, R32.2, R33.2
- new net: D6.2 (A), R33.1
- new net: D5.1 (K), R30.1, U2.12 (OUTA)
- new net: J15.1 (In), R41.1
- new net: J9.1 (In), R21.2
- new net 12V_CM1: FB1.1, L6.2
- new net 12V_CM2: FB2.1, L13.2
- new net C_NTC1: J5.10 (Pin_10), L7.4
- new net C_RTN_12V1: J5.7 (Pin_7), L6.4
- new net C_RTN_12V2: J14.7 (Pin_7), L13.4
- new net C_RTN_DIS1: J5.5 (Pin_5), L5.1
- new net C_RTN_DIS2: J14.5 (Pin_5), L12.1
- new net C_RTN_NTC1: J5.9 (Pin_9), L7.1
- new net C_RTN_PWMH1: J5.1 (Pin_1), L3.1
- new net C_RTN_PWMH2: J14.1 (Pin_1), L10.1
- new net C_RTN_PWML1: J5.3 (Pin_3), L4.4
- new net C_RTN_PWML2: J14.3 (Pin_3), L11.4
- no-connect marks 6 -> 4
Other:
- note added: "Block suffix 1/2 on every driver-side net (GNDI1, VDDA2, ...). Control side (CTRLx 2 x 5 header): PWM_H, PWM_L, DIS, 12 V and (block 1) NTC each with their own return C_RTN_* through one WE-CNSW common-mode choke per pair; 12 V then through a ferrite bead. The control side is a top-layer-only area with a 1200 V barrier (4 mm outer, 3 mm L2) to all power copper; see reports/pcb-rules/PCB_rules_and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"
- note added: "DC link present LED, R49 100 k bleeder"
- note added: "J12 / L8: HS block 2"
- note added: "J13 / L9: LS block 2"
- note added: "J21: AC output, M6 bolt pad, 12 x 5 mm Cu bar bolted on"
- note added: "NTC on the control side (board temperature at the driver)"
- note removed: "Block suffix 1/2 on every driver-side net (GNDI1, VDDA2, ...). Primary side: GNDIx and +12Vx come from the control header through a common-mode choke per pair (12 V/GND, PWM_H/PWM_L, DIS)."
- note removed: "DC link present LED, R50 100 k bleeder"
- note removed: "J12 / L6: HS block 2"
- note removed: "J13 / L7: LS block 2"
- note removed: "J22: AC output, M6 bolt pad, 12 x 5 mm Cu bar bolted on"
- note removed: "J23 is in the LS domain (high voltage)"
- note removed: "NTC on the heatsink side, DC- referenced:"
- moved on the sheet: C22, C24, C25, C26, C56, C58, C59, C60, D6, D7, D8, J16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

Commit message: Rev B boards: 0.5 mm bare-pad rule for the 75 V nets, all 0402 parts to 0603
- New DRC rule: bare pads of different power nets >= 0.5 mm on the outer layers
  (IPC-2221B A6), EPC2361 land pattern and shunt IN land excepted. Bank row A 0.25 mm
  up (was 0.30 mm to row B), top bypass row 0.1 mm towards the bank (0.45 mm to the
  HS gate pads).
- All 0402 resistors/capacitors (and the NTC) are now 0603 for hand soldering; driver
  input side, R_OFF/diode, bottom-side decoupling and U.FL resistors re-placed.
  External PWM pull-downs and the 12 V 4.7 uF dropped (internal 150 k pull-downs;
  12 V only feeds VDDI through 3 k).
- DRC 0/0 and schematic = PCB on both boards; fab outputs and renders regenerated.

Co-Authored-By: Claude Opus 5.5 <noreply@anthropic.com>
Parts:
- removed C87, C88: 22uF 100V X7S 2220, spb_fab:C_2220_5750Metric_TightCrtYd, symbol Device:C
- removed R46: 953R 1%, Resistor_SMD:R_0402_1005Metric, symbol Device:R
- removed R47, R48: 68k, Resistor_SMD:R_1206_3216Metric, symbol Device:R
- removed R49: 100k, Resistor_SMD:R_1206_3216Metric, symbol Device:R
- C13, C14, C15, C16, C47, C48, C49: footprint Capacitor_SMD:C_0402_1005Metric -> Capacitor_SMD:C_0603_1608Metric; MPN Murata GRM155R71C105KA12 -> Murata GRM188R71C105KA12
- C17, C18, C51: footprint Capacitor_SMD:C_0402_1005Metric -> Capacitor_SMD:C_0603_1608Metric; MPN Murata GRM1555C1H101JA01 -> Murata GRM1885C1H101JA01
- C19: footprint Capacitor_SMD:C_0402_1005Metric -> Capacitor_SMD:C_0603_1608Metric; MPN Murata GRM155R71E223KA61 -> Murata GRM188R71E223KA01
- C26, C60: value 4.7uF 25V X5R -> 1uF 100V X7S; footprint Capacitor_SMD:C_0603_1608Metric -> spb_fab:C_0805_2012Metric_TightCrtYd; MPN Murata GRM188R61E475KE11 -> TDK C2012X7S2A105K125AB
- C46: value 1uF 100V X7S -> 1uF 16V X7R; footprint spb_fab:C_0805_2012Metric_TightCrtYd -> Capacitor_SMD:C_0603_1608Metric; MPN TDK C2012X7S2A105K125AB -> Murata GRM188R71C105KA12
- C50: value 1uF 16V X7R -> 100pF C0G; footprint Capacitor_SMD:C_0402_1005Metric -> Capacitor_SMD:C_0603_1608Metric; MPN Murata GRM155R71C105KA12 -> Murata GRM1885C1H101JA01
- C52: value 100pF C0G -> 22nF 25V X7R; footprint Capacitor_SMD:C_0402_1005Metric -> Capacitor_SMD:C_0603_1608Metric; MPN Murata GRM1555C1H101JA01 -> Murata GRM188R71E223KA01
- C53: value 22nF 25V X7R -> 4.7uF 25V X7R; footprint Capacitor_SMD:C_0402_1005Metric -> Capacitor_SMD:C_0805_2012Metric; MPN Murata GRM155R71E223KA61 -> Murata GRM21BR71E475KA73
- C54, C57: value 4.7uF 25V X7R -> 4.7uF 16V X5R; footprint Capacitor_SMD:C_0805_2012Metric -> Capacitor_SMD:C_0603_1608Metric; MPN Murata GRM21BR71E475KA73 -> Murata GRM188R61C475KAAJ
- C56: value 4.7uF 16V X5R -> 4.7uF 25V X7R; footprint Capacitor_SMD:C_0603_1608Metric -> Capacitor_SMD:C_0805_2012Metric; MPN Murata GRM188R61C475KAAJ -> Murata GRM21BR71E475KA73
- C59: value 4.7uF 16V X5R -> 1uF 100V X7S; footprint Capacitor_SMD:C_0603_1608Metric -> spb_fab:C_0805_2012Metric_TightCrtYd; MPN Murata GRM188R61C475KAAJ -> TDK C2012X7S2A105K125AB
- C67, C68: value 1uF 100V X7S -> 22uF 100V X7S 2220; footprint spb_fab:C_0805_2012Metric_TightCrtYd -> spb_fab:C_2220_5750Metric_TightCrtYd; MPN TDK C2012X7S2A105K125AB -> TDK C5750X7S2A226M280KB
- R1, R2, R24, R25, R3, R4: footprint Resistor_SMD:R_0402_1005Metric -> Resistor_SMD:R_0603_1608Metric; MPN 0.5R 0402 1% (Panasonic ERJ-2BQFR50X) -> 0.5R 0603 1% (Panasonic ERJ-3BQFR50V)
- R10, R31, R8: footprint Resistor_SMD:R_0402_1005Metric -> Resistor_SMD:R_0603_1608Metric; MPN 0R 0402 jumper (set R_OFF here) -> 0R 0603 jumper (set R_OFF here)
- R11, R12: footprint Resistor_SMD:R_0402_1005Metric -> Resistor_SMD:R_0603_1608Metric; MPN 47R 0402 1% -> 47R 0603 1%
- R13: footprint Resistor_SMD:R_0402_1005Metric -> Resistor_SMD:R_0603_1608Metric; MPN 3.0k 0402 1% -> 3.0k 0603 1%
- R16, R17, R40: value 10k -> 0R; footprint Resistor_SMD:R_0402_1005Metric -> Resistor_SMD:R_0603_1608Metric; MPN 10k 0402 1% -> 0R 0603
- R18, R21, R42: value 0R -> 953R 1%; footprint Resistor_SMD:R_0402_1005Metric -> Resistor_SMD:R_0603_1608Metric; MPN 0R 0402 -> 953R 0603 1% (75 V working)
- R19, R41: footprint Resistor_SMD:R_0402_1005Metric -> Resistor_SMD:R_0603_1608Metric; MPN 0R 0402 -> 0R 0603
- R20: value 953R 1% -> 0R; footprint Resistor_SMD:R_0402_1005Metric -> Resistor_SMD:R_0603_1608Metric; MPN 953R 0402 1% 100 V -> 0R 0603
- R22: value 0R -> 0R5 1%; footprint Resistor_SMD:R_0402_1005Metric -> Resistor_SMD:R_0603_1608Metric; MPN 0R 0402 -> 0.5R 0603 1% (Panasonic ERJ-3BQFR50V)
- R23: value 953R 1% -> 0R5 1%; footprint Resistor_SMD:R_0402_1005Metric -> Resistor_SMD:R_0603_1608Metric; MPN 953R 0402 1% 100 V -> 0.5R 0603 1% (Panasonic ERJ-3BQFR50V)
- R26, R27: value 0R5 1% -> 10k 1%; footprint Resistor_SMD:R_0402_1005Metric -> Resistor_SMD:R_0603_1608Metric; MPN 0.5R 0402 1% (Panasonic ERJ-2BQFR50X) -> 10k 0603 1%
- R28: value 10k 1% -> 0R75 1%; footprint Resistor_SMD:R_0402_1005Metric -> Resistor_SMD:R_0603_1608Metric; MPN 10k 0402 1% -> 0.75R 0603 1% (Panasonic ERJ-3RQFR75V)
- R29: value 10k 1% -> 0R; footprint Resistor_SMD:R_0402_1005Metric -> Resistor_SMD:R_0603_1608Metric; MPN 10k 0402 1% -> 0R 0603 jumper (set R_OFF here)
- R32: value 0R75 1% -> 47R 1%; MPN 0.75R 0603 1% (Panasonic ERJ-3RQFR75V) -> 47R 0603 1%
- R33: value 0R -> 47R 1%; footprint Resistor_SMD:R_0402_1005Metric -> Resistor_SMD:R_0603_1608Metric; MPN 0R 0402 jumper (set R_OFF here) -> 47R 0603 1%
- R34: value 47R 1% -> 3k 1%; footprint Resistor_SMD:R_0402_1005Metric -> Resistor_SMD:R_0603_1608Metric; MPN 47R 0402 1% -> 3.0k 0603 1%
- R35: value 47R 1% -> 150R 1%; footprint Resistor_SMD:R_0402_1005Metric -> Resistor_SMD:R_0603_1608Metric; MPN 47R 0402 1% -> 150R 0603 1% 0.1 W
- R36: value 3k 1% -> 150R 1%; footprint Resistor_SMD:R_0402_1005Metric -> Resistor_SMD:R_0603_1608Metric; MPN 3.0k 0402 1% -> 150R 0603 1% 0.1 W
- R37, R38: value 150R 1% -> 0R; MPN 150R 0603 1% 0.1 W -> 0R 0603
- R39: value 10k -> 953R 1%; footprint Resistor_SMD:R_0402_1005Metric -> Resistor_SMD:R_0603_1608Metric; MPN 10k 0402 1% -> 953R 0603 1% (75 V working)
- R43: value 953R 1% -> 68k; footprint Resistor_SMD:R_0402_1005Metric -> Resistor_SMD:R_1206_3216Metric; MPN 953R 0402 1% 100 V -> 68k 1206 1% 200 V
- R44: value 0R -> 68k; footprint Resistor_SMD:R_0402_1005Metric -> Resistor_SMD:R_1206_3216Metric; MPN 0R 0402 -> 68k 1206 1% 200 V
- R45: value 0R -> 100k; footprint Resistor_SMD:R_0402_1005Metric -> Resistor_SMD:R_1206_3216Metric; MPN 0R 0402 -> 100k 1206 1% 200 V
- R5, R6: footprint Resistor_SMD:R_0402_1005Metric -> Resistor_SMD:R_0603_1608Metric; MPN 10k 0402 1% -> 10k 0603 1%
- RT1: footprint Resistor_SMD:R_0402_1005Metric -> Resistor_SMD:R_0603_1608Metric; MPN Murata NCP15XH103F03RC -> Murata NCP18XH103F03RB
Connections:
- net +12V1: no longer C26.2
- net +12V2: now also R34.1; no longer C60.2, R36.1
- net DCN: now also C26.1, C34.2, C59.1, C60.1, R45.2; no longer C34.1, C46.2
- net DCP: now also C26.2, C34.1, C59.2, C60.2, R43.1, R45.1; no longer C34.2, C46.1
- net GH_L1: now also R16.2; no longer R18.2
- net GH_L2: now also R22.1, R37.2; no longer R24.1, R41.2
- net GH_R1: now also R19.1; no longer R21.1
- net GH_R2: now also R23.2, R40.1; no longer R25.2, R44.1
- net GL_L1: now also R17.2; no longer R19.2
- net GL_L2: now also R24.1, R38.2; no longer R26.1, R42.2
- net GL_R1: now also R20.1; no longer R22.1
- net GL_R2: now also R25.2, R41.1; no longer R27.2, R45.1
- net GNDI1: now also C18.1, C19.1; no longer C18.2, C19.2, C26.1, R16.2, R17.1
- net GNDI2: now also C50.1, C52.1; no longer C52.2, C53.2, C60.1, R39.2, R40.1
- net KH2: now also C46.1, C54.1, C55.2, R26.1, R35.2; no longer C48.1, C55.1, C56.2, R28.1, R37.2
- net KL1: now also C15.1, C16.1; no longer C15.2, C16.2
- net KL2: now also C48.1, C49.1, C57.2, C58.1, R27.2, R36.2; no longer C49.2, C50.2, C58.2, C59.1, R29.2, R38.2
- net PWM_H1: no longer R16.1
- net PWM_H2: now also R32.1; no longer R34.1, R39.1
- net PWM_L1: no longer R17.2
- net PWM_L2: now also R33.1; no longer R35.1, R40.2
- net SW: now also R18.2, R21.1, R39.2, R42.1; no longer R20.2, R23.1, R43.2
- net VDDA2: now also C46.2, C53.2; no longer C47.2, C55.2
- net VDDB1: now also C16.2; no longer C16.1
- net VDDB2: now also C49.2, C56.2, C58.2; no longer C50.1, C57.2, C59.2
- net VEEA2: now also C47.2, C53.1, C55.1, R35.1; no longer C48.2, C54.1, C56.1, R37.1
- net VEEB1: now also C15.2; no longer C15.1
- net VEEB2: now also C48.2, C56.1, R36.1; no longer C49.1, C58.1, R38.1
- net at R18.1: now also J8.1 (In); no longer J6.1 (In)
- net at R31.1: now also D6.2 (A); no longer D5.2 (A)
- net at R24.2, R25.1, R30.2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: now also R27.1; no longer R28.2
- net at D6.1 (K), U2.9 (OUTB): now also R30.1; no longer R32.1
- net at J17.1 (In): now also R39.1; no longer R43.1
- net at R12.2, U1.3 (INB): now also C18.2; no longer C18.1
- net at R13.2, U1.7 (VDDI): now also C19.2; no longer C19.1
- net at D5.1 (K), U2.12 (OUTA): now also R28.1; no longer R30.1
- net at J20.1 (In): now also R42.2
- net at J16.1 (In): now also R38.1; no longer R42.1
- net at D9.2 (A): now also R44.2
- net at J19.1 (In): now also R41.2; no longer R45.2
- net at J7.1 (In): now also R17.1; no longer R19.1
- net at J15.1 (In): now also R37.1; no longer R41.1
- net at J11.1 (In): now also R21.2; no longer R23.2
- net at R22.2: now also R23.1, R26.2, R28.2, R29.2; no longer J10.1 (In)
- net at J18.1 (In): now also R40.2; no longer R44.2
- net at J9.1 (In): now also R19.2; no longer R21.2
- new net: C50.2, R32.2, U2.2 (INA)
- new net: R43.2, R44.1
- new net: D5.2 (A), R29.1
- new net: C52.2, R34.2, U2.7 (VDDI)
- new net: J6.1 (In), R16.1
- new net: C51.2, R33.2, U2.3 (INB)
- new net: J10.1 (In), R20.2
Other:
- note added: "DC link present LED, R45 100 k bleeder"
- note removed: "DC link present LED, R49 100 k bleeder"
- moved on the sheet: C15, C16, C18, C19, C26, C27, C28, C29, C30, C31, C32, C33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

Commit message: Rev B boards: V_DS port as a 4.99 k 2512 divider (100:1 into 50 R)
- R18/R21/R39/R42: 4.99 k 1 % 2512 (Vishay CRCW25124K99FKEGHP, 1.5 W);
  1.1 W at 75 V into the 50 R scope input, ~0.75 V at the U.FL, so the
  V_DS U.FL is back to U.FL-R-SMT-1(10).
- 2512 on the bottom SW pour under the AC column; 50 R side routed to the
  U.FL through the DC- via-row gap.
- Schematic note and PCB rules document updated.
- DRC 0/0 and schematic = PCB on both boards; fab outputs and renders
  regenerated.

Co-Authored-By: Claude Opus 5.5 <noreply@anthropic.com>
Parts:
- R18, R21, R39, R42: value 953R 1% -> 0R; footprint Resistor_SMD:R_0603_1608Metric -> Resistor_SMD:R_2512_6332Metric; MPN 953R 0603 1% (75 V working) -> Vishay CRCW25124K99FKEGHP (2512, 1.5 W; 1.1 W at 75 V)
Other:
- note added: "U.FL MEASUREMENT PORTS (bottom side, at each cell): V_GS HS / LS (0 R, shield = Kelvin), V_DS LS (4.99 k 2512 series into the 50 R scope input = 100:1, 1.1 W at 75 V; shield = LS source = DC-)"
- note removed: "U.FL MEASUREMENT PORTS (bottom side, at each cell): V_GS HS / LS (0 R, shield = Kelvin), V_DS LS (953 R series = 20:1 into the 50 R scope input, shield = LS source = DC-)"
Changed lines of the file:
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@@
  (text "J12 / L8: HS block 2" (at 439.42 314.96 0) (effects (font (size 1.50 1.50)) (justify left bottom)))
  (text "J13 / L9: LS block 2" (at 642.62 314.96 0) (effects (font (size 1.50 1.50)) (justify left bottom)))
- (text "U.FL MEASUREMENT PORTS (bottom side, at each cell): V_GS HS / LS (0 R, shield = Kelvin), V_DS LS (953 R series = 20:1 into the 50 R scope input, shield = LS source = DC-)" (at 25.40 325.12 0) (effects (font (size 2.00 2.00) bold) (justify left bottom)))
+ (text "U.FL MEASUREMENT PORTS (bottom side, at each cell): V_GS HS / LS (0 R, shield = Kelvin), V_DS LS (4.99 k 2512 series into the 50 R scope input = 100:1, 1.1 W at 75 V; shield = LS source = DC-)" (at 25.40 325.12 0) (effects (font (size 2.00 2.00) bold) (justify left bottom)))
  (text "MOUNTING: H1-H4 board corners (insulated), H5-H7 heatsink spreader; heatsink HS1 (Fischer LAM 4, 100 mm, rotated 90 deg, tube across the board width) is a board-only item" (at 25.40 383.54 0) (effects (font (size 2.00 2.00) bold) (justify left bottom)))
  (text "Nets: DCP = DC+, DCN = DC-, SW = joined switch node of all four cells.  KH1/KH2 and KL1/KL2 are the Kelvin source nets (pad 2 of each EPC2361); they meet the power source only inside the package." (at 25.40 414.02 0) (effects (font (size 1.50 1.50)) (justify left bottom)))
@@
  (symbol (lib_id "Device:R") (at 259.08 337.82 270) (unit 1) (in_bom yes) (on_board yes) (dnp no)
   (property "Reference" "R18" (at 259.08 335.02 90) (effects (font (size 1.27 1.27))))
-  (property "Value" "953R 1%" (at 259.08 340.62 90) (effects (font (size 1.27 1.27))))
-  (property "Footprint" "Resistor_SMD:R_0603_1608Metric" (at 259.08 337.82 90) (effects (font (size 1.27 1.27)) hide))
+  (property "Value" "0R" (at 259.08 340.62 90) (effects (font (size 1.27 1.27))))
+  (property "Footprint" "Resistor_SMD:R_2512_6332Metric" (at 259.08 337.82 90) (effects (font (size 1.27 1.27)) hide))
   (property "Datasheet" "~" (at 259.08 337.82 90) (effects (font (size 1.27 1.27)) hide))
-  (property "MPN" "953R 0603 1% (75 V working)" (at 259.08 337.82 90) (effects (font (size 1.27 1.27)) hide))
-  (property "Description" "953R 1% (V_DS LS, 20:1 into 50 R)" (at 259.08 337.82 90) (effects (font (size 1.27 1.27)) hide))
+  (property "MPN" "Vishay CRCW25124K99FKEGHP (2512, 1.5 W; 1.1 W at 75 V)" (at 259.08 337.82 90) (effects (font (size 1.27 1.27)) hide))
+  (property "Description" "0R (V_DS LS, high-Z probe)" (at 259.08 337.82 90) (effects (font (size 1.27 1.27)) hide))
   (pin "1") (pin "2")
   (instances (project "spb-bb-revb-load" (path "/dd891789-2ead-5ae5-a23c-dd96d7d1b1c9" (reference "R18") (unit 1)))))
@@
  (symbol (lib_id "Device:R") (at 563.88 337.82 90) (unit 1) (in_bom yes) (on_board yes) (dnp no)
   (property "Reference" "R21" (at 563.88 335.02 90) (effects (font (size 1.27 1.27))))
-  (property "Value" "953R 1%" (at 563.88 340.62 90) (effects (font (size 1.27 1.27))))
-  (property "Footprint" "Resistor_SMD:R_0603_1608Metric" (at 563.88 337.82 90) (effects (font (size 1.27 1.27)) hide))
+  (property "Value" "0R" (at 563.88 340.62 90) (effects (font (size 1.27 1.27))))
+  (property "Footprint" "Resistor_SMD:R_2512_6332Metric" (at 563.88 337.82 90) (effects (font (size 1.27 1.27)) hide))
   (property "Datasheet" "~" (at 563.88 337.82 90) (effects (font (size 1.27 1.27)) hide))
-  (property "MPN" "953R 0603 1% (75 V working)" (at 563.88 337.82 90) (effects (font (size 1.27 1.27)) hide))
-  (property "Description" "953R 1% (V_DS LS, 20:1 into 50 R)" (at 563.88 337.82 90) (effects (font (size 1.27 1.27)) hide))
+  (property "MPN" "Vishay CRCW25124K99FKEGHP (2512, 1.5 W; 1.1 W at 75 V)" (at 563.88 337.82 90) (effects (font (size 1.27 1.27)) hide))
+  (property "Description" "0R (V_DS LS, high-Z probe)" (at 563.88 337.82 90) (effects (font (size 1.27 1.27)) hide))
   (pin "1") (pin "2")
   (instances (project "spb-bb-revb-load" (path "/dd891789-2ead-5ae5-a23c-dd96d7d1b1c9" (reference "R21") (unit 1)))))
@@
  (symbol (lib_id "Device:R") (at 259.08 363.22 270) (unit 1) (in_bom yes) (on_board yes) (dnp no)
   (property "Reference" "R39" (at 259.08 360.42 90) (effects (font (size 1.27 1.27))))
-  (property "Value" "953R 1%" (at 259.08 366.02 90) (effects (font (size 1.27 1.27))))
-  (property "Footprint" "Resistor_SMD:R_0603_1608Metric" (at 259.08 363.22 90) (effects (font (size 1.27 1.27)) hide))
+  (property "Value" "0R" (at 259.08 366.02 90) (effects (font (size 1.27 1.27))))
+  (property "Footprint" "Resistor_SMD:R_2512_6332Metric" (at 259.08 363.22 90) (effects (font (size 1.27 1.27)) hide))
   (property "Datasheet" "~" (at 259.08 363.22 90) (effects (font (size 1.27 1.27)) hide))
-  (property "MPN" "953R 0603 1% (75 V working)" (at 259.08 363.22 90) (effects (font (size 1.27 1.27)) hide))
-  (property "Description" "953R 1% (V_DS LS, 20:1 into 50 R)" (at 259.08 363.22 90) (effects (font (size 1.27 1.27)) hide))
+  (property "MPN" "Vishay CRCW25124K99FKEGHP (2512, 1.5 W; 1.1 W at 75 V)" (at 259.08 363.22 90) (effects (font (size 1.27 1.27)) hide))
+  (property "Description" "0R (V_DS LS, high-Z probe)" (at 259.08 363.22 90) (effects (font (size 1.27 1.27)) hide))
   (pin "1") (pin "2")
   (instances (project "spb-bb-revb-load" (path "/dd891789-2ead-5ae5-a23c-dd96d7d1b1c9" (reference "R39") (unit 1)))))
@@
  (symbol (lib_id "Device:R") (at 563.88 363.22 90) (unit 1) (in_bom yes) (on_board yes) (dnp no)
   (property "Reference" "R42" (at 563.88 360.42 90) (effects (font (size 1.27 1.27))))
-  (property "Value" "953R 1%" (at 563.88 366.02 90) (effects (font (size 1.27 1.27))))
-  (property "Footprint" "Resistor_SMD:R_0603_1608Metric" (at 563.88 363.22 90) (effects (font (size 1.27 1.27)) hide))
+  (property "Value" "0R" (at 563.88 366.02 90) (effects (font (size 1.27 1.27))))
+  (property "Footprint" "Resistor_SMD:R_2512_6332Metric" (at 563.88 363.22 90) (effects (font (size 1.27 1.27)) hide))
   (property "Datasheet" "~" (at 563.88 363.22 90) (effects (font (size 1.27 1.27)) hide))
-  (property "MPN" "953R 0603 1% (75 V working)" (at 563.88 363.22 90) (effects (font (size 1.27 1.27)) hide))
-  (property "Description" "953R 1% (V_DS LS, 20:1 into 50 R)" (at 563.88 363.22 90) (effects (font (size 1.27 1.27)) hide))
+  (property "MPN" "Vishay CRCW25124K99FKEGHP (2512, 1.5 W; 1.1 W at 75 V)" (at 563.88 363.22 90) (effects (font (size 1.27 1.27)) hide))
+  (property "Description" "0R (V_DS LS, high-Z probe)" (at 563.88 363.22 90) (effects (font (size 1.27 1.27)) hide))
   (pin "1") (pin "2")
   (instances (project "spb-bb-revb-load" (path "/dd891789-2ead-5ae5-a23c-dd96d7d1b1c9" (reference "R42") (unit 1)))))
