File: PCB-Design/hardware/spb-bb-revb-load/spb-bb-revb-load.kicad_sch (KiCad schematic)
At the start: 194 parts, among them J1 DC+, J10 U.FL L2, J11 U.FL D2, J12 V_ISO,HS in, J13 V_ISO,LS in, J14 CTRL2, J15 U.FL H3, J16 U.FL L3, J17 U.FL D3, J18 U.FL H4, J19 U.FL L4, J2 DC-, J20 U.FL D4, J21 AC, J3 V_ISO,HS in, J4 V_ISO,LS in, J5 CTRL1, J6 U.FL H1, J7 U.FL L1, J8 U.FL D1, J9 U.FL H2, Q1 EPC2361, Q2 EPC2361, Q3 EPC2361, Q4 EPC2361, Q5 EPC2361, Q6 EPC2361, Q7 EPC2361, Q8 EPC2361, U1 2EDF7275K, U2 2EDF7275K

Commit message: Rev B boards: driver output-side 1 uF bypass to 25 V (TDK C1608X7R1E105K080AB)
C13-C16 / C46-C49 (VDD-Kelvin and Kelvin-VEE of each driver output, at most
5.1 V and ~4 V): the 16 V Murata GRM188R71C105KA12D is end of life. Same 0603
footprint, 25 V X7R keeps more of its 1 uF under the DC bias. DRC 0/0 and
schematic = PCB on both boards; fab outputs rebuilt.

Co-Authored-By: Claude Opus 5.5 <noreply@anthropic.com>
Parts:
- C13, C14, C15, C16, C46, C47, C48, C49: MPN Murata GRM188R71C105KA12 -> TDK C1608X7R1E105K080AB
Changed lines of the file:
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@@
   (property "Footprint" "Capacitor_SMD:C_0603_1608Metric" (at 123.19 281.94 0) (effects (font (size 1.27 1.27)) hide))
   (property "Datasheet" "~" (at 123.19 281.94 0) (effects (font (size 1.27 1.27)) hide))
-  (property "MPN" "Murata GRM188R71C105KA12" (at 123.19 281.94 0) (effects (font (size 1.27 1.27)) hide))
+  (property "MPN" "TDK C1608X7R1E105K080AB" (at 123.19 281.94 0) (effects (font (size 1.27 1.27)) hide))
   (property "Description" "1uF 16V X7R 0603" (at 123.19 281.94 0) (effects (font (size 1.27 1.27)) hide))
   (pin "1") (pin "2")
@@
   (property "Footprint" "Capacitor_SMD:C_0603_1608Metric" (at 123.19 297.18 0) (effects (font (size 1.27 1.27)) hide))
   (property "Datasheet" "~" (at 123.19 297.18 0) (effects (font (size 1.27 1.27)) hide))
-  (property "MPN" "Murata GRM188R71C105KA12" (at 123.19 297.18 0) (effects (font (size 1.27 1.27)) hide))
+  (property "MPN" "TDK C1608X7R1E105K080AB" (at 123.19 297.18 0) (effects (font (size 1.27 1.27)) hide))
   (property "Description" "1uF 16V X7R 0603" (at 123.19 297.18 0) (effects (font (size 1.27 1.27)) hide))
   (pin "1") (pin "2")
@@
   (property "Footprint" "Capacitor_SMD:C_0603_1608Metric" (at 326.39 297.18 0) (effects (font (size 1.27 1.27)) hide))
   (property "Datasheet" "~" (at 326.39 297.18 0) (effects (font (size 1.27 1.27)) hide))
-  (property "MPN" "Murata GRM188R71C105KA12" (at 326.39 297.18 0) (effects (font (size 1.27 1.27)) hide))
+  (property "MPN" "TDK C1608X7R1E105K080AB" (at 326.39 297.18 0) (effects (font (size 1.27 1.27)) hide))
   (property "Description" "1uF 16V X7R 0603" (at 326.39 297.18 0) (effects (font (size 1.27 1.27)) hide))
   (pin "1") (pin "2")
@@
   (property "Footprint" "Capacitor_SMD:C_0603_1608Metric" (at 326.39 281.94 0) (effects (font (size 1.27 1.27)) hide))
   (property "Datasheet" "~" (at 326.39 281.94 0) (effects (font (size 1.27 1.27)) hide))
-  (property "MPN" "Murata GRM188R71C105KA12" (at 326.39 281.94 0) (effects (font (size 1.27 1.27)) hide))
+  (property "MPN" "TDK C1608X7R1E105K080AB" (at 326.39 281.94 0) (effects (font (size 1.27 1.27)) hide))
   (property "Description" "1uF 16V X7R 0603" (at 326.39 281.94 0) (effects (font (size 1.27 1.27)) hide))
   (pin "1") (pin "2")
@@
   (property "Footprint" "Capacitor_SMD:C_0603_1608Metric" (at 529.59 281.94 0) (effects (font (size 1.27 1.27)) hide))
   (property "Datasheet" "~" (at 529.59 281.94 0) (effects (font (size 1.27 1.27)) hide))
-  (property "MPN" "Murata GRM188R71C105KA12" (at 529.59 281.94 0) (effects (font (size 1.27 1.27)) hide))
+  (property "MPN" "TDK C1608X7R1E105K080AB" (at 529.59 281.94 0) (effects (font (size 1.27 1.27)) hide))
   (property "Description" "1uF 16V X7R 0603" (at 529.59 281.94 0) (effects (font (size 1.27 1.27)) hide))
   (pin "1") (pin "2")
@@
   (property "Footprint" "Capacitor_SMD:C_0603_1608Metric" (at 529.59 297.18 0) (effects (font (size 1.27 1.27)) hide))
   (property "Datasheet" "~" (at 529.59 297.18 0) (effects (font (size 1.27 1.27)) hide))
-  (property "MPN" "Murata GRM188R71C105KA12" (at 529.59 297.18 0) (effects (font (size 1.27 1.27)) hide))
+  (property "MPN" "TDK C1608X7R1E105K080AB" (at 529.59 297.18 0) (effects (font (size 1.27 1.27)) hide))
   (property "Description" "1uF 16V X7R 0603" (at 529.59 297.18 0) (effects (font (size 1.27 1.27)) hide))
   (pin "1") (pin "2")
@@
   (property "Footprint" "Capacitor_SMD:C_0603_1608Metric" (at 732.79 297.18 0) (effects (font (size 1.27 1.27)) hide))
   (property "Datasheet" "~" (at 732.79 297.18 0) (effects (font (size 1.27 1.27)) hide))
-  (property "MPN" "Murata GRM188R71C105KA12" (at 732.79 297.18 0) (effects (font (size 1.27 1.27)) hide))
+  (property "MPN" "TDK C1608X7R1E105K080AB" (at 732.79 297.18 0) (effects (font (size 1.27 1.27)) hide))
   (property "Description" "1uF 16V X7R 0603" (at 732.79 297.18 0) (effects (font (size 1.27 1.27)) hide))
   (pin "1") (pin "2")
@@
   (property "Footprint" "Capacitor_SMD:C_0603_1608Metric" (at 732.79 281.94 0) (effects (font (size 1.27 1.27)) hide))
   (property "Datasheet" "~" (at 732.79 281.94 0) (effects (font (size 1.27 1.27)) hide))
-  (property "MPN" "Murata GRM188R71C105KA12" (at 732.79 281.94 0) (effects (font (size 1.27 1.27)) hide))
+  (property "MPN" "TDK C1608X7R1E105K080AB" (at 732.79 281.94 0) (effects (font (size 1.27 1.27)) hide))
   (property "Description" "1uF 16V X7R 0603" (at 732.79 281.94 0) (effects (font (size 1.27 1.27)) hide))
   (pin "1") (pin "2")

Commit message: Rev B boards: V_DS U.FL directly on the switch node; pad map regenerated with the board
- V_DS LS ports: the 4.99 k 2512 divider is removed (its 50 R side ran
  ~15 mm over switch-node copper, ~2 pF -> volts of injected error). The
  centre pin sits on the switch node, shield on LSRC; DPT only, 1 MOhm scope
  input, never 50 R. U.FL-R-SMT-1(01) (100 V listed) for these ports.
  The connector's own pin-to-shield gap is excepted from the 0.5 mm rule;
  bottom silk: "VDS U.FL = 75 V: 1 MOHM SCOPE INPUT ONLY".
- The generator now writes pad_nets.json itself. It had not been refreshed
  since 2026-10-16 13:53, so the schematics and the schematic check of the
  later commits ran on a stale pad map; both boards now check against the
  real board data: 0 problems.

Co-Authored-By: Claude Opus 5.5 <noreply@anthropic.com>
Parts:
- removed R42: 0R, Resistor_SMD:R_2512_6332Metric, symbol Device:R
- removed R43, R44: 68k, Resistor_SMD:R_1206_3216Metric, symbol Device:R
- removed R45: 100k, Resistor_SMD:R_1206_3216Metric, symbol Device:R
- C13, C14, C15, C16, C46, C47, C48, C49: value 1uF 16V X7R -> 1uF 25V X7R
- J11, J17, J20, J8: MPN Hirose U.FL-R-SMT-1(10) -> Hirose U.FL-R-SMT-1(01) - 100 V listed, confirm
- R18: footprint Resistor_SMD:R_2512_6332Metric -> Resistor_SMD:R_0603_1608Metric; MPN Vishay CRCW25124K99FKEGHP (2512, 1.5 W; 1.1 W at 75 V) -> 0R 0603
- R20: value 0R -> 0R5 1%; MPN 0R 0603 -> 0.5R 0603 1% (Panasonic ERJ-3BQFR50V)
- R21: value 0R -> 0R5 1%; footprint Resistor_SMD:R_2512_6332Metric -> Resistor_SMD:R_0603_1608Metric; MPN Vishay CRCW25124K99FKEGHP (2512, 1.5 W; 1.1 W at 75 V) -> 0.5R 0603 1% (Panasonic ERJ-3BQFR50V)
- R24, R25: value 0R5 1% -> 10k 1%; MPN 0.5R 0603 1% (Panasonic ERJ-3BQFR50V) -> 10k 0603 1%
- R26: value 10k 1% -> 0R75 1%; MPN 10k 0603 1% -> 0.75R 0603 1% (Panasonic ERJ-3RQFR75V)
- R27: value 10k 1% -> 0R; MPN 10k 0603 1% -> 0R 0603 jumper (set R_OFF here)
- R30: value 0R75 1% -> 47R 1%; MPN 0.75R 0603 1% (Panasonic ERJ-3RQFR75V) -> 47R 0603 1%
- R31: value 0R -> 47R 1%; MPN 0R 0603 jumper (set R_OFF here) -> 47R 0603 1%
- R32: value 47R 1% -> 3k 1%; MPN 47R 0603 1% -> 3.0k 0603 1%
- R33: value 47R 1% -> 150R 1%; MPN 47R 0603 1% -> 150R 0603 1% 0.1 W
- R34: value 3k 1% -> 150R 1%; MPN 3.0k 0603 1% -> 150R 0603 1% 0.1 W
- R35, R36: value 150R 1% -> 0R; MPN 150R 0603 1% 0.1 W -> 0R 0603
- R39: value 0R -> 68k; footprint Resistor_SMD:R_2512_6332Metric -> Resistor_SMD:R_1206_3216Metric; MPN Vishay CRCW25124K99FKEGHP (2512, 1.5 W; 1.1 W at 75 V) -> 68k 1206 1% 200 V
- R40: value 0R -> 68k; footprint Resistor_SMD:R_0603_1608Metric -> Resistor_SMD:R_1206_3216Metric; MPN 0R 0603 -> 68k 1206 1% 200 V
- R41: value 0R -> 100k; footprint Resistor_SMD:R_0603_1608Metric -> Resistor_SMD:R_1206_3216Metric; MPN 0R 0603 -> 100k 1206 1% 200 V
Connections:
- net +12V2: now also R32.1; no longer R34.1
- net DCN: now also R41.2
- net DCP: now also R39.1, R41.1
- net GH_L2: now also R20.1, R35.2; no longer R22.1, R37.2
- net GH_R1: now also R18.1; no longer R19.1
- net GH_R2: now also R21.2, R37.1; no longer R23.2, R40.1
- net GL_L2: now also R22.1, R36.2; no longer R24.1, R38.2
- net GL_R1: now also R19.1; no longer R20.1
- net GL_R2: now also R23.2, R38.1; no longer R25.2, R41.1
- net KH2: now also R24.1, R33.2; no longer R26.1, R35.2
- net KL2: now also R25.2, R34.2; no longer R27.2, R36.2
- net PWM_H2: now also R30.1; no longer R32.1
- net PWM_L2: now also R31.1; no longer R33.1
- net SW: now also J11.1 (In), J17.1 (In), J20.1 (In), J8.1 (In); no longer R18.2, R21.1, R39.2
- net VEEA2: now also R33.1; no longer R35.1
- net VEEB2: now also R34.1; no longer R36.1
- net at D6.2 (A): now also R29.1; no longer R31.1
- net at C50.2, U2.2 (INA): now also R30.2; no longer R32.2
- net at D6.1 (K), U2.9 (OUTB): now also R28.1; no longer R30.1
- net at D5.2 (A): now also R27.1; no longer R29.1
- net at R22.2, R23.1, R28.2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: now also R25.1; no longer R26.2
- net at D5.1 (K), U2.12 (OUTA): now also R26.1; no longer R28.1
- net at J16.1 (In): now also R36.1; no longer R38.1
- net at C52.2, U2.7 (VDDI): now also R32.2; no longer R34.2
- net at D9.2 (A): now also R40.2
- net at C51.2, U2.3 (INB): now also R31.2; no longer R33.2
- net at J15.1 (In): now also R35.1; no longer R37.1
- net at R20.2: now also R21.1, R24.2, R26.2, R27.2; no longer J10.1 (In)
- net at J19.1 (In): now also R38.2; no longer R41.2
- net at J18.1 (In): now also R37.2; no longer R40.2
- net at J9.1 (In): now also R18.2; no longer R19.2
- new net: R39.2, R40.1
- new net: J10.1 (In), R19.2
Other:
- note added: "DC link present LED, R41 100 k bleeder"
- note added: "U.FL MEASUREMENT PORTS (bottom side, at each cell): V_GS HS / LS (0 R, shield = Kelvin), V_DS LS (centre pin directly on the switch node, 1 MOhm scope input only - never 50 R at 75 V; shield = LS source = DC-)"
- note removed: "DC link present LED, R45 100 k bleeder"
- note removed: "U.FL MEASUREMENT PORTS (bottom side, at each cell): V_GS HS / LS (0 R, shield = Kelvin), V_DS LS (4.99 k 2512 series into the 50 R scope input = 100:1, 1.1 W at 75 V; shield = LS source = DC-)"
- moved on the sheet: R18, R19, R20, R21, R22, R23, R24, R25, R26, R27, R28, R29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
