File: PCB-Design/hardware/spb-bb-revb-dpt/spb-bb-revb-dpt.kicad_sch (KiCad schematic)
At the start: 195 parts, among them J1 DC+, J10 U.FL L2, J11 U.FL D2, J12 V_ISO,HS in, J13 V_ISO,LS in, J14 CTRL2, J15 U.FL H3, J16 U.FL L3, J17 U.FL D3, J18 U.FL H4, J19 U.FL L4, J2 DC-, J20 U.FL D4, J21 AC, J3 V_ISO,HS in, J4 V_ISO,LS in, J5 CTRL1, J6 U.FL H1, J7 U.FL L1, J8 U.FL D1, J9 U.FL H2, Q1 EPC2361, Q2 EPC2361, Q3 EPC2361, Q4 EPC2361, Q5 EPC2361, Q6 EPC2361, Q7 EPC2361, Q8 EPC2361, U1 2EDF7275K, U2 2EDF7275K

Commit message: Rev B boards: driver output-side 1 uF bypass to 25 V (TDK C1608X7R1E105K080AB)
C13-C16 / C46-C49 (VDD-Kelvin and Kelvin-VEE of each driver output, at most
5.1 V and ~4 V): the 16 V Murata GRM188R71C105KA12D is end of life. Same 0603
footprint, 25 V X7R keeps more of its 1 uF under the DC bias. DRC 0/0 and
schematic = PCB on both boards; fab outputs rebuilt.

Co-Authored-By: Claude Opus 5.5 <noreply@anthropic.com>
Parts:
- C13, C14, C15, C16, C46, C47, C48, C49: MPN Murata GRM188R71C105KA12 -> TDK C1608X7R1E105K080AB
Changed lines of the file:
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@@
   (property "Footprint" "Capacitor_SMD:C_0603_1608Metric" (at 123.19 281.94 0) (effects (font (size 1.27 1.27)) hide))
   (property "Datasheet" "~" (at 123.19 281.94 0) (effects (font (size 1.27 1.27)) hide))
-  (property "MPN" "Murata GRM188R71C105KA12" (at 123.19 281.94 0) (effects (font (size 1.27 1.27)) hide))
+  (property "MPN" "TDK C1608X7R1E105K080AB" (at 123.19 281.94 0) (effects (font (size 1.27 1.27)) hide))
   (property "Description" "1uF 16V X7R 0603" (at 123.19 281.94 0) (effects (font (size 1.27 1.27)) hide))
   (pin "1") (pin "2")
@@
   (property "Footprint" "Capacitor_SMD:C_0603_1608Metric" (at 123.19 297.18 0) (effects (font (size 1.27 1.27)) hide))
   (property "Datasheet" "~" (at 123.19 297.18 0) (effects (font (size 1.27 1.27)) hide))
-  (property "MPN" "Murata GRM188R71C105KA12" (at 123.19 297.18 0) (effects (font (size 1.27 1.27)) hide))
+  (property "MPN" "TDK C1608X7R1E105K080AB" (at 123.19 297.18 0) (effects (font (size 1.27 1.27)) hide))
   (property "Description" "1uF 16V X7R 0603" (at 123.19 297.18 0) (effects (font (size 1.27 1.27)) hide))
   (pin "1") (pin "2")
@@
   (property "Footprint" "Capacitor_SMD:C_0603_1608Metric" (at 326.39 297.18 0) (effects (font (size 1.27 1.27)) hide))
   (property "Datasheet" "~" (at 326.39 297.18 0) (effects (font (size 1.27 1.27)) hide))
-  (property "MPN" "Murata GRM188R71C105KA12" (at 326.39 297.18 0) (effects (font (size 1.27 1.27)) hide))
+  (property "MPN" "TDK C1608X7R1E105K080AB" (at 326.39 297.18 0) (effects (font (size 1.27 1.27)) hide))
   (property "Description" "1uF 16V X7R 0603" (at 326.39 297.18 0) (effects (font (size 1.27 1.27)) hide))
   (pin "1") (pin "2")
@@
   (property "Footprint" "Capacitor_SMD:C_0603_1608Metric" (at 326.39 281.94 0) (effects (font (size 1.27 1.27)) hide))
   (property "Datasheet" "~" (at 326.39 281.94 0) (effects (font (size 1.27 1.27)) hide))
-  (property "MPN" "Murata GRM188R71C105KA12" (at 326.39 281.94 0) (effects (font (size 1.27 1.27)) hide))
+  (property "MPN" "TDK C1608X7R1E105K080AB" (at 326.39 281.94 0) (effects (font (size 1.27 1.27)) hide))
   (property "Description" "1uF 16V X7R 0603" (at 326.39 281.94 0) (effects (font (size 1.27 1.27)) hide))
   (pin "1") (pin "2")
@@
   (property "Footprint" "Capacitor_SMD:C_0603_1608Metric" (at 529.59 281.94 0) (effects (font (size 1.27 1.27)) hide))
   (property "Datasheet" "~" (at 529.59 281.94 0) (effects (font (size 1.27 1.27)) hide))
-  (property "MPN" "Murata GRM188R71C105KA12" (at 529.59 281.94 0) (effects (font (size 1.27 1.27)) hide))
+  (property "MPN" "TDK C1608X7R1E105K080AB" (at 529.59 281.94 0) (effects (font (size 1.27 1.27)) hide))
   (property "Description" "1uF 16V X7R 0603" (at 529.59 281.94 0) (effects (font (size 1.27 1.27)) hide))
   (pin "1") (pin "2")
@@
   (property "Footprint" "Capacitor_SMD:C_0603_1608Metric" (at 529.59 297.18 0) (effects (font (size 1.27 1.27)) hide))
   (property "Datasheet" "~" (at 529.59 297.18 0) (effects (font (size 1.27 1.27)) hide))
-  (property "MPN" "Murata GRM188R71C105KA12" (at 529.59 297.18 0) (effects (font (size 1.27 1.27)) hide))
+  (property "MPN" "TDK C1608X7R1E105K080AB" (at 529.59 297.18 0) (effects (font (size 1.27 1.27)) hide))
   (property "Description" "1uF 16V X7R 0603" (at 529.59 297.18 0) (effects (font (size 1.27 1.27)) hide))
   (pin "1") (pin "2")
@@
   (property "Footprint" "Capacitor_SMD:C_0603_1608Metric" (at 732.79 297.18 0) (effects (font (size 1.27 1.27)) hide))
   (property "Datasheet" "~" (at 732.79 297.18 0) (effects (font (size 1.27 1.27)) hide))
-  (property "MPN" "Murata GRM188R71C105KA12" (at 732.79 297.18 0) (effects (font (size 1.27 1.27)) hide))
+  (property "MPN" "TDK C1608X7R1E105K080AB" (at 732.79 297.18 0) (effects (font (size 1.27 1.27)) hide))
   (property "Description" "1uF 16V X7R 0603" (at 732.79 297.18 0) (effects (font (size 1.27 1.27)) hide))
   (pin "1") (pin "2")
@@
   (property "Footprint" "Capacitor_SMD:C_0603_1608Metric" (at 732.79 281.94 0) (effects (font (size 1.27 1.27)) hide))
   (property "Datasheet" "~" (at 732.79 281.94 0) (effects (font (size 1.27 1.27)) hide))
-  (property "MPN" "Murata GRM188R71C105KA12" (at 732.79 281.94 0) (effects (font (size 1.27 1.27)) hide))
+  (property "MPN" "TDK C1608X7R1E105K080AB" (at 732.79 281.94 0) (effects (font (size 1.27 1.27)) hide))
   (property "Description" "1uF 16V X7R 0603" (at 732.79 281.94 0) (effects (font (size 1.27 1.27)) hide))
   (pin "1") (pin "2")

Commit message: Rev B boards: V_DS U.FL directly on the switch node; pad map regenerated with the board
- V_DS LS ports: the 4.99 k 2512 divider is removed (its 50 R side ran
  ~15 mm over switch-node copper, ~2 pF -> volts of injected error). The
  centre pin sits on the switch node, shield on LSRC; DPT only, 1 MOhm scope
  input, never 50 R. U.FL-R-SMT-1(01) (100 V listed) for these ports.
  The connector's own pin-to-shield gap is excepted from the 0.5 mm rule;
  bottom silk: "VDS U.FL = 75 V: 1 MOHM SCOPE INPUT ONLY".
- The generator now writes pad_nets.json itself. It had not been refreshed
  since 2026-10-16 13:53, so the schematics and the schematic check of the
  later commits ran on a stale pad map; both boards now check against the
  real board data: 0 problems.

Co-Authored-By: Claude Opus 5.5 <noreply@anthropic.com>
Parts:
- removed R42: 0R, Resistor_SMD:R_2512_6332Metric, symbol Device:R
- removed R43, R44: 68k, Resistor_SMD:R_1206_3216Metric, symbol Device:R
- removed R45: 100k, Resistor_SMD:R_1206_3216Metric, symbol Device:R
- C13, C14, C15, C16, C46, C47, C48, C49: value 1uF 16V X7R -> 1uF 25V X7R
- J11, J17, J20, J8: MPN Hirose U.FL-R-SMT-1(10) -> Hirose U.FL-R-SMT-1(01) - 100 V listed, confirm
- R18: footprint Resistor_SMD:R_2512_6332Metric -> Resistor_SMD:R_0603_1608Metric; MPN Vishay CRCW25124K99FKEGHP (2512, 1.5 W; 1.1 W at 75 V) -> 0R 0603
- R20: value 0R -> 0R5 1%; MPN 0R 0603 -> 0.5R 0603 1% (Panasonic ERJ-3BQFR50V)
- R21: value 0R -> 0R5 1%; footprint Resistor_SMD:R_2512_6332Metric -> Resistor_SMD:R_0603_1608Metric; MPN Vishay CRCW25124K99FKEGHP (2512, 1.5 W; 1.1 W at 75 V) -> 0.5R 0603 1% (Panasonic ERJ-3BQFR50V)
- R24, R25: value 0R5 1% -> 10k 1%; MPN 0.5R 0603 1% (Panasonic ERJ-3BQFR50V) -> 10k 0603 1%
- R26: value 10k 1% -> 0R75 1%; MPN 10k 0603 1% -> 0.75R 0603 1% (Panasonic ERJ-3RQFR75V)
- R27: value 10k 1% -> 0R; MPN 10k 0603 1% -> 0R 0603 jumper (set R_OFF here)
- R30: value 0R75 1% -> 47R 1%; MPN 0.75R 0603 1% (Panasonic ERJ-3RQFR75V) -> 47R 0603 1%
- R31: value 0R -> 47R 1%; MPN 0R 0603 jumper (set R_OFF here) -> 47R 0603 1%
- R32: value 47R 1% -> 3k 1%; MPN 47R 0603 1% -> 3.0k 0603 1%
- R33: value 47R 1% -> 150R 1%; MPN 47R 0603 1% -> 150R 0603 1% 0.1 W
- R34: value 3k 1% -> 150R 1%; MPN 3.0k 0603 1% -> 150R 0603 1% 0.1 W
- R35, R36: value 150R 1% -> 0R; MPN 150R 0603 1% 0.1 W -> 0R 0603
- R39: value 0R -> 68k; footprint Resistor_SMD:R_2512_6332Metric -> Resistor_SMD:R_1206_3216Metric; MPN Vishay CRCW25124K99FKEGHP (2512, 1.5 W; 1.1 W at 75 V) -> 68k 1206 1% 200 V
- R40: value 0R -> 68k; footprint Resistor_SMD:R_0603_1608Metric -> Resistor_SMD:R_1206_3216Metric; MPN 0R 0603 -> 68k 1206 1% 200 V
- R41: value 0R -> 100k; footprint Resistor_SMD:R_0603_1608Metric -> Resistor_SMD:R_1206_3216Metric; MPN 0R 0603 -> 100k 1206 1% 200 V
Connections:
- net +12V2: now also R32.1; no longer R34.1
- net DCN: now also R41.2
- net DCP: now also R39.1, R41.1
- net GH_L2: now also R20.1, R35.2; no longer R22.1, R37.2
- net GH_R1: now also R18.1; no longer R19.1
- net GH_R2: now also R21.2, R37.1; no longer R23.2, R40.1
- net GL_L2: now also R22.1, R36.2; no longer R24.1, R38.2
- net GL_R1: now also R19.1; no longer R20.1
- net GL_R2: now also R23.2, R38.1; no longer R25.2, R41.1
- net KH2: now also R24.1, R33.2; no longer R26.1, R35.2
- net KL2: now also R25.2, R34.2; no longer R27.2, R36.2
- net PWM_H2: now also R30.1; no longer R32.1
- net PWM_L2: now also R31.1; no longer R33.1
- net SW: now also J11.1 (In), J17.1 (In), J20.1 (In), J8.1 (In); no longer R18.2, R21.1, R39.2
- net VEEA2: now also R33.1; no longer R35.1
- net VEEB2: now also R34.1; no longer R36.1
- net at R40.2: now also D9.2 (A); no longer J18.1 (In)
- net at C52.2, U2.7 (VDDI): now also R32.2; no longer R34.2
- net at J16.1 (In): now also R36.1; no longer R38.1
- net at J15.1 (In): now also R35.1; no longer R37.1
- net at R22.2, R23.1, R28.2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: now also R25.1; no longer R26.2
- net at C51.2, U2.3 (INB): now also R31.2; no longer R33.2
- net at D5.1 (K), U2.12 (OUTA): now also R26.1; no longer R28.1
- net at D5.2 (A): now also R27.1; no longer R29.1
- net at D6.1 (K), U2.9 (OUTB): now also R28.1; no longer R30.1
- net at D6.2 (A): now also R29.1; no longer R31.1
- net at C50.2, U2.2 (INA): now also R30.2; no longer R32.2
- net at J19.1 (In): now also R38.2; no longer R41.2
- net at R19.2: now also J10.1 (In); no longer J9.1 (In)
- net at R20.2: now also R21.1, R24.2, R26.2, R27.2; no longer J10.1 (In)
- new net: R39.2, R40.1
- new net: J18.1 (In), R37.2
- new net: J9.1 (In), R18.2
Other:
- note added: "DC link present LED, R41 100 k bleeder"
- note added: "U.FL MEASUREMENT PORTS (bottom side, at each cell): V_GS HS / LS (0 R, shield = Kelvin), V_DS LS (centre pin directly on the switch node, 1 MOhm scope input only - never 50 R at 75 V; shield = LS source LSRCx)"
- note removed: "DC link present LED, R45 100 k bleeder"
- note removed: "U.FL MEASUREMENT PORTS (bottom side, at each cell): V_GS HS / LS (0 R, shield = Kelvin), V_DS LS (4.99 k 2512 series into the 50 R scope input = 100:1, 1.1 W at 75 V; shield = LS source LSRCx)"
- moved on the sheet: R18, R19, R20, R21, R22, R23, R24, R25, R26, R27, R28, R29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

Commit message: DPT board: review fixes - MMCX V_DS ports, saved project rules, test points
Fixes from reports/pcb-rules/spb-bb-revb-dpt-review-2026-10-19.md (DPT only):
- V_DS ports: the U.FL (30 V rating) is replaced by Wurth WR-MMCX
  66012102111404 vertical SMT jacks (170 V rms): centre SW, shield LSRCx,
  bottom side next to each LS FET. The shield goes through the LSS via from
  the shunt IN land; ~25 DC- vias per cell are pruned (mirror pairs).
- Project rules written into the .kicad_pro (track / clearance / connection
  0.2 mm, vias 0.45 / 0.25 mm, ring 0.1 mm, mask web 0.1 mm, courtyards).
  A fresh load of the saved project: DRC 0 / 0 / 0.
- Inner planes: unused inner via rings removed and 0.25 mm minimum fill
  width (the 0.1-0.18 mm necks between antipads are gone).
- Driver barrier exception narrowed to pads and pin-escape tracks.
- Bring-up test points and spring-tip probe pads (board-only footprints,
  scripts/test_points.py, list in fab/testpoints.csv); terminal rule refs
  taken from the board; pad_nets.json written by the generator.
- Docs: DPT_measurement_setup.md, measurement slide, mechanical BOM AC ref,
  stale silk plots archived.
Schematic = PCB (0 problems). Load board not updated in this commit.

Co-Authored-By: Claude Opus 5.5 <noreply@anthropic.com>
Parts:
- J10: value U.FL L2 -> U.FL H2
- J11: value U.FL D2 -> U.FL L2; MPN Hirose U.FL-R-SMT-1(01) - 100 V listed, confirm -> Hirose U.FL-R-SMT-1(10)
- J15: value U.FL H3 -> MMCX VDS L3; footprint spb_fab:U.FL_Hirose_U.FL-R-SMT-1_Vertical -> spb_fab:WR-MMCX_Wuerth_66012102111404_Vertical; MPN Hirose U.FL-R-SMT-1(10) -> Wurth 66012102111404 (WR-MMCX PCB SMT jack, vertical, 170 V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
- J16: value U.FL L3 -> U.FL H3
- J17: value U.FL D3 -> U.FL L3; MPN Hirose U.FL-R-SMT-1(01) - 100 V listed, confirm -> Hirose U.FL-R-SMT-1(10)
- J18: value U.FL H4 -> MMCX VDS L4; footprint spb_fab:U.FL_Hirose_U.FL-R-SMT-1_Vertical -> spb_fab:WR-MMCX_Wuerth_66012102111404_Vertical; MPN Hirose U.FL-R-SMT-1(10) -> Wurth 66012102111404 (WR-MMCX PCB SMT jack, vertical, 170 V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
- J19: value U.FL L4 -> U.FL H4
- J20: value U.FL D4 -> U.FL L4; MPN Hirose U.FL-R-SMT-1(01) - 100 V listed, confirm -> Hirose U.FL-R-SMT-1(10)
- J6: value U.FL H1 -> MMCX VDS L1; footprint spb_fab:U.FL_Hirose_U.FL-R-SMT-1_Vertical -> spb_fab:WR-MMCX_Wuerth_66012102111404_Vertical; MPN Hirose U.FL-R-SMT-1(10) -> Wurth 66012102111404 (WR-MMCX PCB SMT jack, vertical, 170 V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
- J7: value U.FL L1 -> U.FL H1
- J8: value U.FL D1 -> U.FL L1; MPN Hirose U.FL-R-SMT-1(01) - 100 V listed, confirm -> Hirose U.FL-R-SMT-1(10)
- J9: value U.FL H2 -> MMCX VDS L2; footprint spb_fab:U.FL_Hirose_U.FL-R-SMT-1_Vertical -> spb_fab:WR-MMCX_Wuerth_66012102111404_Vertical; MPN Hirose U.FL-R-SMT-1(10) -> Wurth 66012102111404 (WR-MMCX PCB SMT jack, vertical, 170 V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
Connections:
- net KH1: now also J10.2 (Ext), J7.2 (Ext); no longer J6.2 (Ext), J9.2 (Ext)
- net KH2: now also J16.2 (Ext), J19.2 (Ext); no longer J15.2 (Ext), J18.2 (Ext)
- net KL1: now also J11.2 (Ext), J8.2 (Ext); no longer J10.2 (Ext), J7.2 (Ext)
- net KL2: now also J17.2 (Ext), J20.2 (Ext); no longer J16.2 (Ext), J19.2 (Ext)
- net LSRC1: now also J6.2 (Ext); no longer J8.2 (Ext)
- net LSRC2: now also J9.2 (Ext); no longer J11.2 (Ext)
- net LSRC3: now also J15.2 (Ext); no longer J17.2 (Ext)
- net LSRC4: now also J18.2 (Ext); no longer J20.2 (Ext)
- net SW: now also J15.1 (In), J18.1 (In), J6.1 (In), J9.1 (In); no longer J11.1 (In), J17.1 (In), J20.1 (In), J8.1 (In)
- net at J7.1 (In): now also R16.1; no longer R17.1
- net at R38.2: now also J20.1 (In); no longer J19.1 (In)
- net at R35.1: now also J16.1 (In); no longer J15.1 (In)
- net at R19.2: now also J11.1 (In); no longer J10.1 (In)
- net at R37.2: now also J19.1 (In); no longer J18.1 (In)
- net at R18.2: now also J10.1 (In); no longer J9.1 (In)
- net at R36.1: now also J17.1 (In); no longer J16.1 (In)
- new net: J8.1 (In), R17.1
Other:
- note added: "MEASUREMENT PORTS (bottom side, at each cell): U.FL V_GS HS / LS (0 R from the gate, shield = Kelvin); MMCX V_DS LS (Wurth WR-MMCX, 170 V rms; centre = SW at the LS drain, shield = LS source LSRCx, device side of the shunt; for a rated isolated probe, e.g. IsoVu TIVP + TIVPMX50X)"
- note removed: "U.FL MEASUREMENT PORTS (bottom side, at each cell): V_GS HS / LS (0 R, shield = Kelvin), V_DS LS (centre pin directly on the switch node, 1 MOhm scope input only - never 50 R at 75 V; shield = LS source LSRCx)"
- moved on the sheet: R16, R17, R18, R19, R35, R36, R37, R38

Commit message: DPT board: fabrication review fixes - gate re-layout, mirrored DC- vias, fab package
- G1/G2: R_G at the gate pad, Kelvin return beside the gate on L1 to the corridor,
  Kelvin rows joined under the star (HS L4, LS L2), point-symmetric about each star
  (the two cells of a row are rotated 180 deg); 10k pull-downs as 0402 between the rows
- G3: 0R U.FL gate-sense links DNP by default
- P1: shunt-return via rows counted from the inner edge, all DC- vias mirrored
- F1/F2: fab notes in the Gerber zip (stack-up, rules, tenting, via-in-pad list),
  separate PTH/NPTH drill files
- F4: BOM grouped by value, RS1-RS4 lab-fitted (not in pick-and-place)
- loop_post: cell-to-cell loop mutual matrix; gate model refs follow the new R_G
- generator QUICK=1 mode (DRC after fill, no test points)
- review document with the dispositions

DRC 0/0 (also fresh load), sch = PCB, no 3D collisions, 36 labelled test points.

Co-Authored-By: Claude Opus 5.5 <noreply@anthropic.com>
Parts:
- R16, R17, R18, R19, R35, R36, R37, R38: value 0R -> DNP 0R; MPN 0R 0603 -> 0R 0603 - not fitted by default
- R22, R3: value 0R5 1% -> 10k 1%; footprint Resistor_SMD:R_0603_1608Metric -> Resistor_SMD:R_0402_1005Metric; MPN 0.5R 0603 1% (Panasonic ERJ-3BQFR50V) -> 10k 0402 1%
- R24, R5: value 10k 1% -> 0R5 1%; MPN 10k 0603 1% -> 0.5R 0603 1% (Panasonic ERJ-3BQFR50V)
- R25, R6: footprint Resistor_SMD:R_0603_1608Metric -> Resistor_SMD:R_0402_1005Metric; MPN 10k 0603 1% -> 10k 0402 1%
Connections:
- net GL_L1: now also R4.1; no longer R3.1
- net GL_L2: now also R23.1; no longer R22.1
- net GL_R1: now also R5.2; no longer R4.2
- net GL_R2: now also R24.2; no longer R23.2
- net KH1: now also R3.2; no longer R5.1
- net KH2: now also R22.2; no longer R24.1
- net at R20.2, R21.1, R26.2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: now also R22.1; no longer R24.2
- net at R25.1, R28.2, R29.2: now also R23.2, R24.1; no longer R22.2, R23.1
- net at R1.2, R2.1, R7.2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: now also R3.1; no longer R5.2
- net at R10.2, R6.1, R9.2: now also R4.2, R5.1; no longer R3.2, R4.1
Other:
- moved on the sheet: R22, R23, R24, R3, R4, R5
