File: PCB-Design/hardware/spb-bb-revb-dpt/spb-bb-revb-dpt.kicad_sch (KiCad schematic)
At the start: 191 parts, among them J1 DC+, J10 U.FL H2, J11 U.FL L2, J12 V_ISO,HS in, J13 V_ISO,LS in, J14 CTRL2, J15 MMCX VDS L3, J16 U.FL H3, J17 U.FL L3, J18 MMCX VDS L4, J19 U.FL H4, J2 DC-, J20 U.FL L4, J21 AC, J3 V_ISO,HS in, J4 V_ISO,LS in, J5 CTRL1, J6 MMCX VDS L1, J7 U.FL H1, J8 U.FL L1, J9 MMCX VDS L2, Q1 EPC2361, Q2 EPC2361, Q3 EPC2361, Q4 EPC2361, Q5 EPC2361, Q6 EPC2361, Q7 EPC2361, Q8 EPC2361, U1 2EDF7275K, U2 2EDF7275K

Commit message: DPT board: R_ON 1.0 Ohm (R_G,on 2.5 Ohm per device)
- R7/R9/R26/R28 0.75 -> 1.0 Ohm (Yageo RC0603FR-071RL): with the extracted gate
  network the HS V_DS peak at the LS turn-on drops from 100.0 V to 93.7 V (75 V, 322 A),
  E_on 105 uJ (= design-flow value), cell spread E_on 0.2 %, I_off +-2.2 % (inner vs outer
  cells, power side)
- SPICE: sweep varies R_ON with R_G fixed at 0.5 Ohm (R_G = R_G,on - 2 R_ON went to 0);
  block 2 is block 1 shifted, not mirrored (cell 3 <-> 1, 4 <-> 2); the 1.25 Ohm case
  diverged numerically and is dropped
- DRC 0/0 (fresh load too), sch = PCB, no 3D collisions, 36 test points

Co-Authored-By: Claude Opus 5.5 <noreply@anthropic.com>
Parts:
- R26, R28, R7, R9: value 0R75 1% -> 1R0 1%; MPN 0.75R 0603 1% (Panasonic ERJ-3RQFR75V) -> 1.0R 0603 1% (Yageo RC0603FR-071RL)
Other:
- note added: "R_ON 1.0 R, R_OFF 0 R (jumper), R_G 0.5 R per transistor, 10 k gate pull-down at the star to the Kelvin net"
- note removed: "R_ON 0.75 R, R_OFF 0 R (jumper), R_G 0.5 R per transistor, 10 k gate pull-down at the star to the Kelvin net"
Changed lines of the file:
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@@
  (text "NTC on the control side (board temperature at the driver)" (at 33.02 262.89 0) (effects (font (size 1.27 1.27)) (justify left bottom)))
  (text "SLDON = GNDI: input-side LDO on" (at 139.70 248.92 0) (effects (font (size 1.27 1.27)) (justify left bottom)))
- (text "R_ON 0.75 R, R_OFF 0 R (jumper), R_G 0.5 R per transistor, 10 k gate pull-down at the star to the Kelvin net" (at 139.70 251.46 0) (effects (font (size 1.27 1.27)) (justify left bottom)))
+ (text "R_ON 1.0 R, R_OFF 0 R (jumper), R_G 0.5 R per transistor, 10 k gate pull-down at the star to the Kelvin net" (at 139.70 251.46 0) (effects (font (size 1.27 1.27)) (justify left bottom)))
  (text "BLOCK 2" (at 436.88 190.50 0) (effects (font (size 1.80 1.80) bold) (justify left bottom)))
  (text "SLDON = GNDI: input-side LDO on" (at 546.10 248.92 0) (effects (font (size 1.27 1.27)) (justify left bottom)))
- (text "R_ON 0.75 R, R_OFF 0 R (jumper), R_G 0.5 R per transistor, 10 k gate pull-down at the star to the Kelvin net" (at 546.10 251.46 0) (effects (font (size 1.27 1.27)) (justify left bottom)))
+ (text "R_ON 1.0 R, R_OFF 0 R (jumper), R_G 0.5 R per transistor, 10 k gate pull-down at the star to the Kelvin net" (at 546.10 251.46 0) (effects (font (size 1.27 1.27)) (justify left bottom)))
  (text "GATE SUPPLY ISLANDS: external isolated supply (one HS, one LS, split per block) -> WE-CNSW -> 5.1 V Zener VDD-S, 150 R bias S-VEE: V_GS,on = +5.1 V, V_GS,off = -(V_ISO - 5.1 V)" (at 25.40 266.70 0) (effects (font (size 2.00 2.00) bold) (justify left bottom)))
  (text "J3 / L1: HS block 1" (at 33.02 314.96 0) (effects (font (size 1.50 1.50)) (justify left bottom)))
@@
  (symbol (lib_id "Device:R") (at 604.52 215.90 90) (unit 1) (in_bom yes) (on_board yes) (dnp no)
   (property "Reference" "R26" (at 604.52 213.10 90) (effects (font (size 1.27 1.27))))
-  (property "Value" "0R75 1%" (at 604.52 218.70 90) (effects (font (size 1.27 1.27))))
+  (property "Value" "1R0 1%" (at 604.52 218.70 90) (effects (font (size 1.27 1.27))))
   (property "Footprint" "Resistor_SMD:R_0603_1608Metric" (at 604.52 215.90 90) (effects (font (size 1.27 1.27)) hide))
   (property "Datasheet" "~" (at 604.52 215.90 90) (effects (font (size 1.27 1.27)) hide))
-  (property "MPN" "0.75R 0603 1% (Panasonic ERJ-3RQFR75V)" (at 604.52 215.90 90) (effects (font (size 1.27 1.27)) hide))
-  (property "Description" "0R75 1% (R_ON,A)" (at 604.52 215.90 90) (effects (font (size 1.27 1.27)) hide))
+  (property "MPN" "1.0R 0603 1% (Yageo RC0603FR-071RL)" (at 604.52 215.90 90) (effects (font (size 1.27 1.27)) hide))
+  (property "Description" "1R0 1% (R_ON,A)" (at 604.52 215.90 90) (effects (font (size 1.27 1.27)) hide))
   (pin "1") (pin "2")
   (instances (project "spb-bb-revb-dpt" (path "/e62a99d0-4c10-5aed-840f-6353566af670" (reference "R26") (unit 1)))))
@@
  (symbol (lib_id "Device:R") (at 604.52 226.06 90) (unit 1) (in_bom yes) (on_board yes) (dnp no)
   (property "Reference" "R28" (at 604.52 223.26 90) (effects (font (size 1.27 1.27))))
-  (property "Value" "0R75 1%" (at 604.52 228.86 90) (effects (font (size 1.27 1.27))))
+  (property "Value" "1R0 1%" (at 604.52 228.86 90) (effects (font (size 1.27 1.27))))
   (property "Footprint" "Resistor_SMD:R_0603_1608Metric" (at 604.52 226.06 90) (effects (font (size 1.27 1.27)) hide))
   (property "Datasheet" "~" (at 604.52 226.06 90) (effects (font (size 1.27 1.27)) hide))
-  (property "MPN" "0.75R 0603 1% (Panasonic ERJ-3RQFR75V)" (at 604.52 226.06 90) (effects (font (size 1.27 1.27)) hide))
-  (property "Description" "0R75 1% (R_ON,B)" (at 604.52 226.06 90) (effects (font (size 1.27 1.27)) hide))
+  (property "MPN" "1.0R 0603 1% (Yageo RC0603FR-071RL)" (at 604.52 226.06 90) (effects (font (size 1.27 1.27)) hide))
+  (property "Description" "1R0 1% (R_ON,B)" (at 604.52 226.06 90) (effects (font (size 1.27 1.27)) hide))
   (pin "1") (pin "2")
   (instances (project "spb-bb-revb-dpt" (path "/e62a99d0-4c10-5aed-840f-6353566af670" (reference "R28") (unit 1)))))
@@
  (symbol (lib_id "Device:R") (at 198.12 215.90 90) (unit 1) (in_bom yes) (on_board yes) (dnp no)
   (property "Reference" "R7" (at 198.12 213.10 90) (effects (font (size 1.27 1.27))))
-  (property "Value" "0R75 1%" (at 198.12 218.70 90) (effects (font (size 1.27 1.27))))
+  (property "Value" "1R0 1%" (at 198.12 218.70 90) (effects (font (size 1.27 1.27))))
   (property "Footprint" "Resistor_SMD:R_0603_1608Metric" (at 198.12 215.90 90) (effects (font (size 1.27 1.27)) hide))
   (property "Datasheet" "~" (at 198.12 215.90 90) (effects (font (size 1.27 1.27)) hide))
-  (property "MPN" "0.75R 0603 1% (Panasonic ERJ-3RQFR75V)" (at 198.12 215.90 90) (effects (font (size 1.27 1.27)) hide))
-  (property "Description" "0R75 1% (R_ON,A)" (at 198.12 215.90 90) (effects (font (size 1.27 1.27)) hide))
+  (property "MPN" "1.0R 0603 1% (Yageo RC0603FR-071RL)" (at 198.12 215.90 90) (effects (font (size 1.27 1.27)) hide))
+  (property "Description" "1R0 1% (R_ON,A)" (at 198.12 215.90 90) (effects (font (size 1.27 1.27)) hide))
   (pin "1") (pin "2")
   (instances (project "spb-bb-revb-dpt" (path "/e62a99d0-4c10-5aed-840f-6353566af670" (reference "R7") (unit 1)))))
@@
  (symbol (lib_id "Device:R") (at 198.12 226.06 90) (unit 1) (in_bom yes) (on_board yes) (dnp no)
   (property "Reference" "R9" (at 198.12 223.26 90) (effects (font (size 1.27 1.27))))
-  (property "Value" "0R75 1%" (at 198.12 228.86 90) (effects (font (size 1.27 1.27))))
+  (property "Value" "1R0 1%" (at 198.12 228.86 90) (effects (font (size 1.27 1.27))))
   (property "Footprint" "Resistor_SMD:R_0603_1608Metric" (at 198.12 226.06 90) (effects (font (size 1.27 1.27)) hide))
   (property "Datasheet" "~" (at 198.12 226.06 90) (effects (font (size 1.27 1.27)) hide))
-  (property "MPN" "0.75R 0603 1% (Panasonic ERJ-3RQFR75V)" (at 198.12 226.06 90) (effects (font (size 1.27 1.27)) hide))
-  (property "Description" "0R75 1% (R_ON,B)" (at 198.12 226.06 90) (effects (font (size 1.27 1.27)) hide))
+  (property "MPN" "1.0R 0603 1% (Yageo RC0603FR-071RL)" (at 198.12 226.06 90) (effects (font (size 1.27 1.27)) hide))
+  (property "Description" "1R0 1% (R_ON,B)" (at 198.12 226.06 90) (effects (font (size 1.27 1.27)) hide))
   (pin "1") (pin "2")
   (instances (project "spb-bb-revb-dpt" (path "/e62a99d0-4c10-5aed-840f-6353566af670" (reference "R9") (unit 1)))))
